File: kicad/k1-aioc/k1-aioc.kicad_pcb (KiCad board)
At the start: 2 copper layers, 21 x 31.5 mm, 39 parts, among them J1 12401832E402A, J2 Conn_01x07_Male, Q1 BC847BS, U1 LP2985-3.3, U2 STM32F373CBTx, Y1 8MHz/20pF

Commit message: Cosmetic changes
Routing:
- net GND: vias 70 -> 71

Commit message: Added missing 1.5K USB pullup resistor
Parts:
- added R1: 1.5K, Resistor_SMD:R_0603_1608Metric, F.Cu at (110.8, 92.0)
- moved FB2 0.90 mm to (108.2, 91.5), turned to 90 degrees
- moved C4 0.25 mm to (108.2, 94.5)
- moved C6 0.25 mm to (105.5, 90.8)
- moved U1 0.25 mm to (105.5, 94.0)
Routing:
- net +3V3: track 41.6 -> 46.3 mm, vias 5 -> 6
- net /USB-DP: track 11.7 -> 13.2 mm
- net GND: track 8.99 -> 10.00 mm, vias 71 -> 67
- net /VBUS: track 10.8 -> 11.7 mm
Other:
- board text added: "AIOC Rev. 1 S. Kueppers"
- board text removed: "AIOC Rev. 0 S. Kueppers"

Commit message: Resistor position cleanup
Parts:
- moved R6 0.75 mm to (117.8, 84.0)
- moved R7 0.75 mm to (117.8, 87.0)
Routing:
- net GND: vias 67 -> 69
Changed lines of the file:
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@@
   )
   (footprint "Resistor_SMD:R_0603_1608Metric" (layer "F.Cu")
-    (at 117.75 83.25 -90)
+    (at 117.75 84 -90)
     (descr "Resistor SMD 0603 (1608 Metric), square (rectangular) end terminal, IPC_7351 nominal, (Body size source: IPC-SM-782 page 72, https://www.pcb-3d.com/wordpress/wp-content/uploads/ipc-sm-782a_amendment_1_and_2.pdf), generated with kicad-footprint-generator")
     (tags "resistor")
@@
   )
   (footprint "Resistor_SMD:R_0603_1608Metric" (layer "F.Cu")
-    (at 117.75 86.25 90)
+    (at 117.75 87 90)
     (descr "Resistor SMD 0603 (1608 Metric), square (rectangular) end terminal, IPC_7351 nominal, (Body size source: IPC-SM-782 page 72, https://www.pcb-3d.com/wordpress/wp-content/uploads/ipc-sm-782a_amendment_1_and_2.pdf), generated with kicad-footprint-generator")
     (tags "resistor")
@@
   (via (at 115.5 97.5) (size 0.6) (drill 0.3) (layers "F.Cu" "B.Cu") (net 1))
   (via (at 113 83.5) (size 0.6) (drill 0.3) (layers "F.Cu" "B.Cu") (free) (net 1))
-  (via (at 117.75 81.5) (size 0.6) (drill 0.3) (layers "F.Cu" "B.Cu") (net 1))
   (via (at 105.5 94) (size 0.6) (drill 0.3) (layers "F.Cu" "B.Cu") (net 1))
   (via (at 104.5 109) (size 0.6) (drill 0.3) (layers "F.Cu" "B.Cu") (free) (net 1))
   (via (at 114.242052 88.160946) (size 0.6) (drill 0.3) (layers "F.Cu" "B.Cu") (net 1))
   (via (at 116.5 94.5) (size 0.6) (drill 0.3) (layers "F.Cu" "B.Cu") (net 1))
+  (via (at 118.95 83.25) (size 0.6) (drill 0.3) (layers "F.Cu" "B.Cu") (net 1))
   (via (at 104.5 108) (size 0.6) (drill 0.3) (layers "F.Cu" "B.Cu") (free) (net 1))
   (via (at 115 102) (size 0.6) (drill 0.3) (layers "F.Cu" "B.Cu") (free) (net 1))
@@
   (via (at 113 96.5) (size 0.6) (drill 0.3) (layers "F.Cu" "B.Cu") (free) (net 1))
   (via (at 110 100.25) (size 0.6) (drill 0.3) (layers "F.Cu" "B.Cu") (free) (net 1))
+  (via (at 118.95 84.75) (size 0.6) (drill 0.3) (layers "F.Cu" "B.Cu") (net 1))
   (via (at 109.25 103.75) (size 0.6) (drill 0.3) (layers "F.Cu" "B.Cu") (free) (net 1))
   (via (at 112.25 102) (size 0.6) (drill 0.3) (layers "F.Cu" "B.Cu") (free) (net 1))
@@
   (via (at 115.5 101) (size 0.6) (drill 0.3) (layers "F.Cu" "B.Cu") (free) (net 1))
   (via (at 111.5 102) (size 0.6) (drill 0.3) (layers "F.Cu" "B.Cu") (free) (net 1))
+  (via (at 118.95 86.25) (size 0.6) (drill 0.3) (layers "F.Cu" "B.Cu") (net 1))
   (via (at 109.25 104.75) (size 0.6) (drill 0.3) (layers "F.Cu" "B.Cu") (free) (net 1))
   (via (at 115.5 92) (size 0.6) (drill 0.3) (layers "F.Cu" "B.Cu") (net 1))
-  (via (at 117.75 88) (size 0.6) (drill 0.3) (layers "F.Cu" "B.Cu") (net 1))
+  (via (at 118.95 87.75) (size 0.6) (drill 0.3) (layers "F.Cu" "B.Cu") (net 1))
   (via (at 110 83.5) (size 0.6) (drill 0.3) (layers "F.Cu" "B.Cu") (free) (net 1))
   (segment (start 106.275 109.125) (end 106.15 109.25) (width 0.25) (layer "F.Cu") (net 2))
@@
   (segment (start 111.35 90.380761) (end 111.35 90.5) (width 0.3) (layer "F.Cu") (net 25))
   (segment (start 111.5 87.32) (end 111.5 86.4) (width 0.3) (layer "F.Cu") (net 25))
-  (segment (start 111.5 93.4) (end 111.5 95.0875) (width 0.3) (layer "F.Cu") (net 25))
   (segment (start 111.35 93.25) (end 111.35 92.85) (width 0.25) (layer "F.Cu") (net 25))
-  (segment (start 111.35 93.175) (end 111.35 93.25) (width 0.3) (layer "F.Cu") (net 25))
-  (segment (start 111.325 93.15) (end 111.35 93.175) (width 0.3) (layer "F.Cu") (net 25))
   (segment (start 111.5 86.4) (end 111.35 86.25) (width 0.3) (layer "F.Cu") (net 25))
   (segment (start 111.35 92.85) (end 111.575 92.625) (width 0.25) (layer "F.Cu") (net 25))
+  (segment (start 111.5 95.0875) (end 111.5 93.4) (width 0.3) (layer "F.Cu") (net 25))
   (segment (start 111.75 89.02) (end 111.75 89.980761) (width 0.3) (layer "F.Cu") (net 25))
-  (segment (start 111.35 93.25) (end 111.5 93.4) (width 0.3) (layer "F.Cu") (net 25))
+  (segment (start 111.5 93.4) (end 111.35 93.25) (width 0.3) (layer "F.Cu") (net 25))
   (segment (start 111.75 89.980761) (end 111.35 90.380761) (width 0.3) (layer "F.Cu") (net 25))
   (via (at 111.35 86.25) (size 0.6) (drill 0.3) (layers "F.Cu" "B.Cu") (free) (net 25))
   (via (at 111.35 90.5) (size 0.6) (drill 0.3) (layers "F.Cu" "B.Cu") (free) (net 25))
   (via (at 111.35 93.25) (size 0.6) (drill 0.3) (layers "F.Cu" "B.Cu") (free) (net 25))
-  (segment (start 111.35 93.25) (end 111.4 93.2) (width 0.5) (layer "B.Cu") (net 25))
-  (segment (start 111.4 86.3) (end 111.35 86.25) (width 0.5) (layer "B.Cu") (net 25))
-  (segment (start 111.4 93.2) (end 111.4 86.3) (width 0.5) (layer "B.Cu") (net 25))
+  (segment (start 111.4 86.3) (end 111.4 93.2) (width 0.5) (layer "B.Cu") (net 25))
+  (segment (start 111.35 86.25) (end 111.4 86.3) (width 0.5) (layer "B.Cu") (net 25))
+  (segment (start 111.4 93.2) (end 111.35 93.25) (width 0.5) (layer "B.Cu") (net 25))
+  (segment (start 112 95.0875) (end 112 93.4) (width 0.3) (layer "F.Cu") (net 26))
   (segment (start 110.7 90.769239) (end 111.080761 91.15) (width 0.3) (layer "F.Cu") (net 26))
   (segment (start 112 86.4) (end 112.15 86.25) (width 0.3) (layer "F.Cu") (net 26))
-  (segment (start 112 93.4) (end 112 95.0875) (width 0.3) (layer "F.Cu") (net 26))
   (segment (start 111.619239 91.15) (end 112.15 90.619239) (width 0.3) (layer "F.Cu") (net 26))
   (segment (start 111.080761 91.15) (end 111.619239 91.15) (width 0.3) (layer "F.Cu") (net 26))
-  (segment (start 112.15 93.25) (end 112 93.4) (width 0.3) (layer "F.Cu") (net 26))
   (segment (start 112 87.32) (end 112 86.4) (width 0.3) (layer "F.Cu") (net 26))
   (segment (start 111.25 89.02) (end 111.25 89.680761) (width 0.3) (layer "F.Cu") (net 26))
+  (segment (start 112 93.4) (end 112.15 93.25) (width 0.3) (layer "F.Cu") (net 26))
   (segment (start 110.7 90.230761) (end 110.7 90.769239) (width 0.3) (layer "F.Cu") (net 26))
   (segment (start 111.25 89.680761) (end 110.7 90.230761) (width 0.3) (layer "F.Cu") (net 26))
@@
   (via (at 112.15 90.5) (size 0.6) (drill 0.3) (layers "F.Cu" "B.Cu") (free) (net 26))
   (via (at 112.15 93.25) (size 0.6) (drill 0.3) (layers "F.Cu" "B.Cu") (free) (net 26))
-  (segment (start 112.1 86.3) (end 112.15 86.25) (width 0.5) (layer "B.Cu") (net 26))
-  (segment (start 112.1 93.2) (end 112.1 86.3) (width 0.5) (layer "B.Cu") (net 26))
-  (segment (start 112.15 93.25) (end 112.1 93.2) (width 0.5) (layer "B.Cu") (net 26))
+  (segment (start 112.1 93.2) (end 112.15 93.25) (width 0.5) (layer "B.Cu") (net 26))
+  (segment (start 112.1 86.3) (end 112.1 93.2) (width 0.5) (layer "B.Cu") (net 26))
+  (segment (start 112.15 86.25) (end 112.1 86.3) (width 0.5) (layer "B.Cu") (net 26))
   (segment (start 104.55 95.1375) (end 104.55 95.8) (width 0.5) (layer "F.Cu") (net 27))
   (segment (start 104.55 95.8) (end 104.75 96) (width 0.5) (layer "F.Cu") (net 27))
@@
   (segment (start 117.925 92) (end 117.925 90.55) (width 0.3) (layer "F.Cu") (net 35))
   (segment (start 117.925 90.55) (end 117.975 90.5) (width 0.3) (layer "F.Cu") (net 35))
-  (segment (start 115.75 84.75) (end 111.5 84.75) (width 0.25) (layer "F.Cu") (net 36))
   (segment (start 111 86.783884) (end 111 87.32) (width 0.25) (layer "F.Cu") (net 36))
-  (segment (start 116.925 84.075) (end 116.25 84.75) (width 0.25) (layer "F.Cu") (net 36))
-  (segment (start 117.75 84.075) (end 116.925 84.075) (width 0.25) (layer "F.Cu") (net 36))
+  (segment (start 111.425 84.825) (end 110.725 85.525) (width 0.25) (layer "F.Cu") (net 36))
   (segment (start 110.725 85.525) (end 110.725 86.508884) (width 0.25) (layer "F.Cu") (net 36))
+  (segment (start 117.75 84.825) (end 111.425 84.825) (width 0.25) (layer "F.Cu") (net 36))
   (segment (start 110.725 86.508884) (end 111 86.783884) (width 0.25) (layer "F.Cu") (net 36))
-  (segment (start 116.25 84.75) (end 115.75 84.75) (width 0.25) (layer "F.Cu") (net 36))
-  (segment (start 111.5 84.75) (end 110.725 85.525) (width 0.25) (layer "F.Cu") (net 36))
   (segment (start 112.6495 89.942499) (end 112.25 89.542999) (width 0.25) (layer "F.Cu") (net 37))
   (segment (start 112.25 89.542999) (end 112.25 89.02) (width 0.25) (layer "F.Cu") (net 37))
-  (segment (start 114.075 85.425) (end 113.75 85.75) (width 0.25) (layer "F.Cu") (net 37))
-  (segment (start 118 85.425) (end 114.075 85.425) (width 0.25) (layer "F.Cu") (net 37))
+  (segment (start 114.075 85.425) (end 116.175 85.425) (width 0.25) (layer "F.Cu") (net 37))
+  (segment (start 116.925 86.175) (end 117.75 86.175) (width 0.25) (layer "F.Cu") (net 37))
+  (segment (start 113.75 85.75) (end 114.075 85.425) (width 0.25) (layer "F.Cu") (net 37))
+  (segment (start 116.175 85.425) (end 116.925 86.175) (width 0.25) (layer "F.Cu") (net 37))
   (via (at 113.75 85.75) (size 0.6) (drill 0.3) (layers "F.Cu" "B.Cu") (net 37))
   (via (at 112.8995 89.942499) (size 0.6) (drill 0.3) (layers "F.Cu" "B.Cu") (net 37))

Commit message: Added missing biasing resistor on AFIN
Parts:
- added R16: 5.1K, Resistor_SMD:R_0603_1608Metric, F.Cu at (118.8, 92.0)
- R3: value 2.2K -> 5.1K
- moved C14 3.00 mm to (121.8, 90.5)
- moved R5 1.50 mm to (118.8, 90.5), turned to 0 degrees
Routing:
- net /AFIN: track 8.24 -> 11.1 mm
- net +3.3VA: track 29.2 -> 31.5 mm
- net /RADIO-SPK: track 3.79 -> 2.76 mm

Commit message: Slightly added board shape and added 1mm thru-hole
Parts:
- added H1: MountingHole, TestPoint:TestPoint_THTPad_D2.0mm_Drill1.0mm, F.Cu at (118.2, 81.2)
Other:
- outline, holes or cut-outs redrawn
Changed lines of the file:
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@@
   (net 32 "/VIN")
   (net 33 "/VBUS")
-  (net 34 "Net-(R2-Pad2)")
+  (net 34 "Net-(C12-Pad1)")
   (net 35 "Net-(C14-Pad1)")
   (net 36 "Net-(J1-PadB5)")
@@
       (net 47 "/AFOUT") (pintype "passive"))
     (pad "2" smd roundrect (at 0.825 0 270) (size 0.8 0.95) (layers "F.Cu" "F.Paste" "F.Mask") (roundrect_rratio 0.25)
-      (net 34 "Net-(R2-Pad2)") (pintype "passive"))
+      (net 34 "Net-(C12-Pad1)") (pintype "passive"))
     (model "${KICAD6_3DMODEL_DIR}/Resistor_SMD.3dshapes/R_0603_1608Metric.wrl"
       (offset (xyz 0 0 0))
@@
     (fp_line (start 0.8 0.4) (end -0.8 0.4) (layer "F.Fab") (width 0.1))
     (pad "1" smd roundrect (at -0.775 0) (size 0.9 0.95) (layers "F.Cu" "F.Paste" "F.Mask") (roundrect_rratio 0.25)
-      (net 34 "Net-(R2-Pad2)") (pintype "passive"))
+      (net 34 "Net-(C12-Pad1)") (pintype "passive"))
     (pad "2" smd roundrect (at 0.775 0) (size 0.9 0.95) (layers "F.Cu" "F.Paste" "F.Mask") (roundrect_rratio 0.25)
       (net 1 "GND") (pintype "passive"))
@@
       (net 1 "GND") (pintype "passive"))
     (pad "2" smd roundrect (at 0.825 0 180) (size 0.8 0.95) (layers "F.Cu" "F.Paste" "F.Mask") (roundrect_rratio 0.25)
-      (net 34 "Net-(R2-Pad2)") (pintype "passive"))
+      (net 34 "Net-(C12-Pad1)") (pintype "passive"))
     (model "${KICAD6_3DMODEL_DIR}/Resistor_SMD.3dshapes/R_0603_1608Metric.wrl"
       (offset (xyz 0 0 0))
@@
     )
   )
+  (footprint "TestPoint:TestPoint_THTPad_D2.0mm_Drill1.0mm" (layer "F.Cu")
+    (at 118.25 81.25)
+    (descr "THT pad as test Point, diameter 2.0mm, hole diameter 1.0mm")
+    (tags "test point THT pad")
+    (property "Sheetfile" "k1-aioc.kicad_sch")
+    (property "Sheetname" "")
+    (attr exclude_from_pos_files)
+    (fp_text reference "H1" (at 0 -1.998) (layer "F.SilkS")
+      (effects (font (size 1 1) (thickness 0.15)))
+    )
+    (fp_text value "MountingHole" (at 0 2.05) (layer "F.Fab")
+      (effects (font (size 1 1) (thickness 0.15)))
+    )
+    (fp_text user "${REFERENCE}" (at 0 -2) (layer "F.Fab")
+      (effects (font (size 1 1) (thickness 0.15)))
+    )
+    (fp_circle (center 0 0) (end 0 1.2) (layer "F.SilkS") (width 0.12) (fill none))
+    (fp_circle (center 0 0) (end 1.5 0) (layer "F.CrtYd") (width 0.05) (fill none))
+    (pad "1" thru_hole circle (at 0 0) (size 2 2) (drill 1) (layers *.Cu *.Mask))
+  )
   (footprint "Capacitor_SMD:C_0603_1608Metric" (layer "F.Cu")
     (at 119.5 106.25 -90)
@@
     (fp_line (start 0.8 0.4) (end -0.8 0.4) (layer "F.Fab") (width 0.1))
     (pad "1" smd roundrect (at -0.775 0 270) (size 0.9 0.95) (layers "F.Cu" "F.Paste" "F.Mask") (roundrect_rratio 0.25)
-      (net 34 "Net-(R2-Pad2)") (pintype "passive"))
+      (net 34 "Net-(C12-Pad1)") (pintype "passive"))
     (pad "2" smd roundrect (at 0.775 0 270) (size 0.9 0.95) (layers "F.Cu" "F.Paste" "F.Mask") (roundrect_rratio 0.25)
       (net 45 "/RADIO-MIC") (pintype "passive"))
@@
   (gr_rect (start 124.5 104.25) (end 139.5 108) (layer "Dwgs.User") (width 0.15) (fill none))
   (gr_rect (start 124.5 92.75) (end 139.5 95.25) (layer "Dwgs.User") (width 0.15) (fill none))
-  (gr_line (start 119.5 88.25) (end 119.5 80.5) (layer "Edge.Cuts") (width 0.1))
-  (gr_line (start 103.5 111) (end 103.5 80.5) (layer "Edge.Cuts") (width 0.1))
+  (gr_line (start 119.5 88.25) (end 119.5 81.25) (layer "Edge.Cuts") (width 0.1))
+  (gr_line (start 103.5 110.25) (end 103.5 81.25) (layer "Edge.Cuts") (width 0.1))
   (gr_line (start 120.75 89.5) (end 124 89.5) (layer "Edge.Cuts") (width 0.1))
   (gr_line (start 124.5 90) (end 124.5 111) (layer "Edge.Cuts") (width 0.1))
-  (gr_line (start 124 111.5) (end 104 111.5) (layer "Edge.Cuts") (width 0.1))
+  (gr_line (start 124 111.5) (end 104.75 111.5) (layer "Edge.Cuts") (width 0.1))
   (gr_arc (start 124.5 111) (mid 124.353553 111.353553) (end 124 111.5) (layer "Edge.Cuts") (width 0.1))
   (gr_line (start 120.75 89.5) (end 119.5 88.25) (layer "Edge.Cuts") (width 0.1))
-  (gr_line (start 106 80) (end 119 80) (layer "Edge.Cuts") (width 0.1))
-  (gr_arc (start 119 80) (mid 119.353553 80.146447) (end 119.5 80.5) (layer "Edge.Cuts") (width 0.1))
+  (gr_arc (start 118.25 80) (mid 119.133883 80.366117) (end 119.5 81.25) (layer "Edge.Cuts") (width 0.1))
+  (gr_arc (start 103.5 81.25) (mid 103.866117 80.366117) (end 104.75 80) (layer "Edge.Cuts") (width 0.1))
+  (gr_line (start 106 80) (end 118.25 80) (layer "Edge.Cuts") (width 0.1))
   (gr_arc (start 124 89.5) (mid 124.353553 89.646447) (end 124.5 90) (layer "Edge.Cuts") (width 0.1))
-  (gr_arc (start 104 111.5) (mid 103.646447 111.353553) (end 103.5 111) (layer "Edge.Cuts") (width 0.1))
-  (gr_line (start 106 80) (end 104 80) (layer "Edge.Cuts") (width 0.1))
-  (gr_arc (start 103.5 80.5) (mid 103.646447 80.146447) (end 104 80) (layer "Edge.Cuts") (width 0.1))
+  (gr_line (start 106 80) (end 104.75 80) (layer "Edge.Cuts") (width 0.1))
+  (gr_arc (start 104.75 111.5) (mid 103.866117 111.133883) (end 103.5 110.25) (layer "Edge.Cuts") (width 0.1))
   (gr_text "RST" (at 104.25 82.75 270) (layer "B.SilkS")
     (effects (font (size 0.4 0.4) (thickness 0.1)) (justify mirror))
@@
   (segment (start 112.6 105.122183) (end 112.6 107.4) (width 0.25) (layer "F.Cu") (net 51))
   (via (at 112.6 107.75) (size 0.6) (drill 0.3) (layers "F.Cu" "B.Cu") (net 51))
-  (segment (start 103.85 110.483884) (end 103.85 83.15) (width 0.25) (layer "B.Cu") (net 51))
-  (segment (start 103.85 83.15) (end 104.33 82.67) (width 0.25) (layer "B.Cu") (net 51))
-  (segment (start 112.075 111.125) (end 104.491116 111.125) (width 0.25) (layer "B.Cu") (net 51))
-  (segment (start 104.33 82.67) (end 105.25 82.67) (width 0.25) (layer "B.Cu") (net 51))
-  (segment (start 104.491116 111.125) (end 103.85 110.483884) (width 0.25) (layer "B.Cu") (net 51))
   (segment (start 112.6 110.6) (end 112.075 111.125) (width 0.25) (layer "B.Cu") (net 51))
+  (segment (start 104.725 111.125) (end 103.85 110.25) (width 0.25) (layer "B.Cu") (net 51))
   (segment (start 112.6 107.75) (end 112.6 110.6) (width 0.25) (layer "B.Cu") (net 51))
+  (segment (start 103.85 110.25) (end 103.85 83.15) (width 0.25) (layer "B.Cu") (net 51))
+  (segment (start 103.85 83.15) (end 104.33 82.67) (width 0.25) (layer "B.Cu") (net 51))
+  (segment (start 112.075 111.125) (end 104.725 111.125) (width 0.25) (layer "B.Cu") (net 51))
+  (segment (start 104.33 82.67) (end 105.25 82.67) (width 0.25) (layer "B.Cu") (net 51))
   (segment (start 109.65 97.240685) (end 109.390685 97.5) (width 0.25) (layer "F.Cu") (net 52))
   (segment (start 109.5 96.109315) (end 109.65 96.259315) (width 0.25) (layer "F.Cu") (net 52))
