File: kicad/k1-aioc/k1-aioc.kicad_pcb (KiCad board)
At the start: 2 copper layers, 21 x 31.5 mm, 42 parts, among them J1 12401832E402A, J2 Conn_01x07_Male, Q1 BC847BS, U1 LP2985-3.3, U2 STM32F373CBTx, Y1 8MHz/20pF

Commit message: Added alternative LED footprints on bottom side
Parts:
- added D3: N.M., LED_SMD:LED_0603_1608Metric, B.Cu at (105.5, 103.5)
- added D4: N.M., LED_SMD:LED_0603_1608Metric, B.Cu at (105.5, 105.0)
- D1: value LED -> GREEN
- D2: value LED -> RED
- moved D1 1.50 mm to (105.5, 103.5)
- moved D2 1.50 mm to (105.5, 105.0)
Routing:
- net Net-(D1-Pad2): track 5.48 -> 9.76 mm, vias 0 -> 1
- net Net-(D1-Pad1): track 3.02 -> 7.30 mm, vias 0 -> 1
- net GND: vias 69 -> 68
Changed lines of the file:
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@@
   )
   (footprint "LED_SMD:LED_0603_1608Metric" (layer "F.Cu")
-    (at 105.5 103.5 180)
+    (at 105.5 105 180)
     (descr "LED SMD 0603 (1608 Metric), square (rectangular) end terminal, IPC_7351 nominal, (Body size source: http://www.tortai-tech.com/upload/download/2011102023233369053.pdf), generated with kicad-footprint-generator")
     (tags "LED")
@@
       (effects (font (size 0.5 0.5) (thickness 0.1)))
     )
-    (fp_text value "LED" (at 0 1.43) (layer "F.Fab")
+    (fp_text value "RED" (at 0 1.43) (layer "F.Fab")
       (effects (font (size 1 1) (thickness 0.15)))
     )
@@
   )
   (footprint "LED_SMD:LED_0603_1608Metric" (layer "F.Cu")
-    (at 105.5 105)
+    (at 105.5 103.5)
     (descr "LED SMD 0603 (1608 Metric), square (rectangular) end terminal, IPC_7351 nominal, (Body size source: http://www.tortai-tech.com/upload/download/2011102023233369053.pdf), generated with kicad-footprint-generator")
     (tags "LED")
@@
       (effects (font (size 0.5 0.5) (thickness 0.1)))
     )
-    (fp_text value "LED" (at 0 1.43) (layer "F.Fab")
+    (fp_text value "GREEN" (at 0 1.43) (layer "F.Fab")
       (effects (font (size 1 1) (thickness 0.15)))
     )
@@
     (pad "7" thru_hole oval (at 0 7.62 180) (size 1 1) (drill 0.65) (layers *.Cu *.Mask)
       (net 52 "/SWO") (pinfunction "Pin_7") (pintype "passive"))
-    (model "${KICAD6_3DMODEL_DIR}/Connector_PinHeader_1.27mm.3dshapes/PinHeader_1x07_P1.27mm_Horizontal.wrl"
+    (model "${KICAD6_3DMODEL_DIR}/Connector_PinHeader_1.27mm.3dshapes/PinHeader_1x07_P1.27mm_Horizontal.wrl" hide
       (offset (xyz 0 0 0))
       (scale (xyz 1 1 1))
@@
     )
   )
+  (footprint "LED_SMD:LED_0603_1608Metric" (layer "B.Cu")
+    (at 105.5 105 180)
+    (descr "LED SMD 0603 (1608 Metric), square (rectangular) end terminal, IPC_7351 nominal, (Body size source: http://www.tortai-tech.com/upload/download/2011102023233369053.pdf), generated with kicad-footprint-generator")
+    (tags "LED")
+    (property "LCSC" "")
+    (property "Sheetfile" "k1-aioc.kicad_sch")
+    (property "Sheetname" "")
+    (attr smd exclude_from_pos_files)
+    (fp_text reference "D4" (at 0 1.43) (layer "B.SilkS") hide
+      (effects (font (size 1 1) (thickness 0.15)) (justify mirror))
+    )
+    (fp_text value "N.M." (at 0 -1.43) (layer "B.Fab")
+      (effects (font (size 1 1) (thickness 0.15)) (justify mirror))
+    )
+    (fp_text user "${REFERENCE}" (at 0 0) (layer "B.Fab")
+      (effects (font (size 0.4 0.4) (thickness 0.06)) (justify mirror))
+    )
+    (fp_line (start -1.485 0.735) (end -1.485 -0.735) (layer "B.SilkS") (width 0.12))
+    (fp_line (start -1.485 -0.735) (end 0.8 -0.735) (layer "B.SilkS") (width 0.12))
+    (fp_line (start 0.8 0.735) (end -1.485 0.735) (layer "B.SilkS") (width 0.12))
+    (fp_line (start -1.48 0.73) (end 1.48 0.73) (layer "B.CrtYd") (width 0.05))
+    (fp_line (start 1.48 -0.73) (end -1.48 -0.73) (layer "B.CrtYd") (width 0.05))
+    (fp_line (start 1.48 0.73) (end 1.48 -0.73) (layer "B.CrtYd") (width 0.05))
+    (fp_line (start -1.48 -0.73) (end -1.48 0.73) (layer "B.CrtYd") (width 0.05))
+    (fp_line (start 0.8 -0.4) (end 0.8 0.4) (layer "B.Fab") (width 0.1))
+    (fp_line (start -0.5 0.4) (end -0.8 0.1) (layer "B.Fab") (width 0.1))
+    (fp_line (start -0.8 0.1) (end -0.8 -0.4) (layer "B.Fab") (width 0.1))
+    (fp_line (start -0.8 -0.4) (end 0.8 -0.4) (layer "B.Fab") (width 0.1))
+    (fp_line (start 0.8 0.4) (end -0.5 0.4) (layer "B.Fab") (width 0.1))
+    (pad "1" smd roundrect (at -0.7875 0 180) (size 0.875 0.95) (layers "B.Cu" "B.Paste" "B.Mask") (roundrect_rratio 0.25)
+      (net 55 "Net-(D1-Pad2)") (pinfunction "K") (pintype "passive"))
+    (pad "2" smd roundrect (at 0.7875 0 180) (size 0.875 0.95) (layers "B.Cu" "B.Paste" "B.Mask") (roundrect_rratio 0.25)
+      (net 54 "Net-(D1-Pad1)") (pinfunction "A") (pintype "passive"))
+    (model "${KICAD6_3DMODEL_DIR}/LED_SMD.3dshapes/LED_0603_1608Metric.wrl" hide
+      (offset (xyz 0 0 0))
+      (scale (xyz 1 1 1))
+      (rotate (xyz 0 0 0))
+    )
+  )
   (footprint "Symbol:OSHW-Logo2_7.3x6mm_SilkScreen" (layer "B.Cu")
     (at 108 108.25 180)
@@
       ) (layer "B.SilkS") (width 0.01) (fill solid))
   )
+  (footprint "LED_SMD:LED_0603_1608Metric" (layer "B.Cu")
+    (at 105.5 103.5)
+    (descr "LED SMD 0603 (1608 Metric), square (rectangular) end terminal, IPC_7351 nominal, (Body size source: http://www.tortai-tech.com/upload/download/2011102023233369053.pdf), generated with kicad-footprint-generator")
+    (tags "LED")
+    (property "LCSC" "")
+    (property "Sheetfile" "k1-aioc.kicad_sch")
+    (property "Sheetname" "")
+    (attr smd exclude_from_pos_files)
+    (fp_text reference "D3" (at 0 1.43) (layer "B.SilkS") hide
+      (effects (font (size 1 1) (thickness 0.15)) (justify mirror))
+    )
+    (fp_text value "N.M." (at 0 -1.43) (layer "B.Fab")
+      (effects (font (size 1 1) (thickness 0.15)) (justify mirror))
+    )
+    (fp_text user "${REFERENCE}" (at 0 0) (layer "B.Fab")
+      (effects (font (size 0.4 0.4) (thickness 0.06)) (justify mirror))
+    )
+    (fp_line (start -1.485 -0.735) (end 0.8 -0.735) (layer "B.SilkS") (width 0.12))
+    (fp_line (start 0.8 0.735) (end -1.485 0.735) (layer "B.SilkS") (width 0.12))
+    (fp_line (start -1.485 0.735) (end -1.485 -0.735) (layer "B.SilkS") (width 0.12))
+    (fp_line (start -1.48 0.73) (end 1.48 0.73) (layer "B.CrtYd") (width 0.05))
+    (fp_line (start -1.48 -0.73) (end -1.48 0.73) (layer "B.CrtYd") (width 0.05))
+    (fp_line (start 1.48 -0.73) (end -1.48 -0.73) (layer "B.CrtYd") (width 0.05))
+    (fp_line (start 1.48 0.73) (end 1.48 -0.73) (layer "B.CrtYd") (width 0.05))
+    (fp_line (start 0.8 0.4) (end -0.5 0.4) (layer "B.Fab") (width 0.1))
+    (fp_line (start -0.8 -0.4) (end 0.8 -0.4) (layer "B.Fab") (width 0.1))
+    (fp_line (start 0.8 -0.4) (end 0.8 0.4) (layer "B.Fab") (width 0.1))
+    (fp_line (start -0.5 0.4) (end -0.8 0.1) (layer "B.Fab") (width 0.1))
+    (fp_line (start -0.8 0.1) (end -0.8 -0.4) (layer "B.Fab") (width 0.1))
+    (pad "1" smd roundrect (at -0.7875 0) (size 0.875 0.95) (layers "B.Cu" "B.Paste" "B.Mask") (roundrect_rratio 0.25)
+      (net 54 "Net-(D1-Pad1)") (pinfunction "K") (pintype "passive"))
+    (pad "2" smd roundrect (at 0.7875 0) (size 0.875 0.95) (layers "B.Cu" "B.Paste" "B.Mask") (roundrect_rratio 0.25)
+      (net 55 "Net-(D1-Pad2)") (pinfunction "A") (pintype "passive"))
+    (model "${KICAD6_3DMODEL_DIR}/LED_SMD.3dshapes/LED_0603_1608Metric.wrl" hide
+      (offset (xyz 0 0 0))
+      (scale (xyz 1 1 1))
+      (rotate (xyz 0 0 0))
+    )
+  )
   (gr_rect (start 107.1 86.55) (end 107.65 87.65) (layer "F.Paste") (width 0.3) (fill solid))
   (gr_rect (start 106.75 80.6) (end 107.3 81.7) (layer "F.Paste") (width 0.3) (fill solid))
@@
   (via (at 105.5 94.75) (size 0.6) (drill 0.3) (layers "F.Cu" "B.Cu") (net 1))
   (via (at 121.75 100) (size 0.8) (drill 0.4) (layers "F.Cu" "B.Cu") (free) (net 1))
-  (via (at 105.5 104.25) (size 0.6) (drill 0.3) (layers "F.Cu" "B.Cu") (free) (net 1))
   (via (at 116.5 95.5) (size 0.6) (drill 0.3) (layers "F.Cu" "B.Cu") (net 1))
   (via (at 111.5 110) (size 0.6) (drill 0.3) (layers "F.Cu" "B.Cu") (free) (net 1))
@@
   (segment (start 104.575 100.175) (end 104.325 99.925) (width 0.25) (layer "B.Cu") (net 53))
   (segment (start 104.325 97.325) (end 104.3 97.3) (width 0.25) (layer "B.Cu") (net 53))
+  (segment (start 105.5 105.25) (end 105.5 105.75) (width 0.25) (layer "F.Cu") (net 54))
+  (segment (start 104.7125 105) (end 105.25 105) (width 0.25) (layer "F.Cu") (net 54))
+  (segment (start 105.25 105) (end 105.5 105.25) (width 0.25) (layer "F.Cu") (net 54))
   (segment (start 104.7125 105.05) (end 104.7125 102.0875) (width 0.25) (layer "F.Cu") (net 54))
   (segment (start 104.7125 102.0875) (end 104.675 102.05) (width 0.25) (layer "F.Cu") (net 54))
+  (via (at 105.5 105.75) (size 0.6) (drill 0.3) (layers "F.Cu" "B.Cu") (net 54))
+  (segment (start 104.7125 103.5) (end 104.7125 105) (width 0.25) (layer "B.Cu") (net 54))
+  (segment (start 105.25 105) (end 105.5 105.25) (width 0.25) (layer "B.Cu") (net 54))
+  (segment (start 105.5 105.25) (end 105.5 105.75) (width 0.25) (layer "B.Cu") (net 54))
+  (segment (start 104.7125 105) (end 105.25 105) (width 0.25) (layer "B.Cu") (net 54))
   (segment (start 106.2875 105.05) (end 106.2875 103.55) (width 0.25) (layer "F.Cu") (net 55))
   (segment (start 107.525 102.3125) (end 106.2875 103.55) (width 0.25) (layer "F.Cu") (net 55))
   (segment (start 108.5875 101) (end 107.772792 101) (width 0.25) (layer "F.Cu") (net 55))
   (segment (start 107.772792 101) (end 107.525 101.247792) (width 0.25) (layer "F.Cu") (net 55))
+  (segment (start 105.5 103.75) (end 105.5 104.25) (width 0.25) (layer "F.Cu") (net 55))
+  (segment (start 106.2875 103.5) (end 105.75 103.5) (width 0.25) (layer "F.Cu") (net 55))
   (segment (start 107.525 101.247792) (end 107.525 102.3125) (width 0.25) (layer "F.Cu") (net 55))
+  (segment (start 105.75 103.5) (end 105.5 103.75) (width 0.25) (layer "F.Cu") (net 55))
+  (via (at 105.5 104.25) (size 0.6) (drill 0.3) (layers "F.Cu" "B.Cu") (net 55))
+  (segment (start 106.2875 103.5) (end 106.2875 105) (width 0.25) (layer "B.Cu") (net 55))
+  (segment (start 106.2875 103.5) (end 105.75 103.5) (width 0.25) (layer "B.Cu") (net 55))
+  (segment (start 105.5 103.75) (end 105.5 104.25) (width 0.25) (layer "B.Cu") (net 55))
+  (segment (start 105.75 103.5) (end 105.5 103.75) (width 0.25) (layer "B.Cu") (net 55))
   (segment (start 107.636396 100.5) (end 107.075 101.061396) (width 0.25) (layer "F.Cu") (net 56))
   (segment (start 108.5875 100.5) (end 107.636396 100.5) (width 0.25) (layer "F.Cu") (net 56))

Commit message: Adjusted OSHW logo
Parts:
- removed #LOGO1: OSHW-Logo2_7.3x6mm_SilkScreen, Symbol:OSHW-Logo2_7.3x6mm_SilkScreen
- added REF**: OSHW-Logo2_9.8x8mm_SilkScreen, Symbol:OSHW-Logo2_9.8x8mm_SilkScreen, B.Cu at (112.5, 106.2)
Routing:
- net GND: vias 68 -> 66

Commit message: Replaced single 3.3V LDO by dual 3.3V LDO to suppress 1kHz noise from USB in analog signals
Parts:
- added C5: 4.7u/10V/X5R, Capacitor_SMD:C_0603_1608Metric, F.Cu at (104.8, 98.0)
- C3: value 10n/NP0 -> 100n
- C7: value 100n -> 4.7u/10V/X5R
- C9: value 4.7u/10V/X5R -> 100n
- U1: value LP2985-3.3 -> MIC5330-SSYML; footprint Package_TO_SOT_SMD:SOT-23-5 -> Package_DFN_QFN:Micrel_MLF-8-1EP_2x2mm_P0.5mm_EP0.6x1.2mm
- moved C3 6.25 mm to (104.8, 91.5), turned to 90 degrees
- moved C6 1.06 mm to (106.2, 91.5), turned to 90 degrees
- moved U1 0.75 mm to (105.5, 94.8)
- moved C4 0.50 mm to (107.8, 94.5)
- moved FB2 0.50 mm to (107.8, 91.5)
- moved FB1 0.25 mm to (106.2, 98.0), turned to 90 degrees
- moved J2 0.25 mm to (105.2, 88.8)
Connections:
- FB1 pad 1: +3V3 -> +3.3VA
- FB1 pad 2: +3.3VA -> Net-(U1-Pad7)
- U1 pad 3: /VIN -> Net-(C3-Pad1)
- U1 pad 4: Net-(C3-Pad1) -> /VIN
- U1 pad 5: +3V3 -> /VIN
- U2 pad 1: unconnected-(U2-Pad1) -> +3V3
Routing:
- net /VIN: track 6.95 -> 11.5 mm
- net Net-(U1-Pad7): track 0.00 -> 3.11 mm
- net GND: track 10.00 -> 7.84 mm, vias 66 -> 60
- net +3V3: track 46.3 -> 47.9 mm, vias 6 -> 5

Commit message: Modified board shape to be narrower at TRS connector end
Parts:
- moved C11 1.50 mm to (118.8, 92.0)
- moved C14 1.50 mm to (121.8, 92.0)
- moved R16 1.50 mm to (118.8, 93.5)
- moved C12 0.50 mm to (121.2, 103.5)
- moved C7 0.50 mm to (119.8, 100.5)
- moved R2 0.50 mm to (119.0, 102.8)
- moved R4 0.50 mm to (121.2, 102.0)
- moved R6 0.25 mm to (117.8, 84.2)
- moved R7 0.25 mm to (117.8, 87.2)
Routing:
- net /RADIO-RX-PTT1: track 26.9 -> 30.0 mm
- net /RADIO-TX: track 26.6 -> 24.2 mm
- net Net-(C14-Pad1): track 1.40 -> 2.48 mm
- net /RADIO-SPK: track 2.76 -> 2.01 mm
- net +3.3VA: track 31.4 -> 30.8 mm
- net Net-(C12-Pad1): track 5.63 -> 5.13 mm
- net GND: vias 60 -> 61
Other:
- outline, holes or cut-outs redrawn

Commit message: Modified placement of programming header
Parts:
- moved J2 0.33 mm to (104.9, 88.8)
