File: kicad/k1-aioc/k1-aioc.kicad_pcb (KiCad board)
At the start: 2 copper layers, 21 x 31.5 mm, 45 parts, among them J1 12401832E402A, J2 Conn_01x07_Male, Q1 BC847BS, U1 MIC5330-SSYML, U2 STM32F373CBTx, Y1 8MHz/20pF

Commit message: Adjusted bottom side silkscreen
Parts:
- moved R6 0.25 mm to (117.8, 84.5)
- moved R7 0.25 mm to (117.8, 87.5)
Routing:
- net GND: vias 61 -> 60
Other:
- board text added: "AIOC V1.0"
- board text added: "S. Kueppers"
- board text removed: "AIOC Rev. 1 S. Kueppers"

Commit message: Rotated SWD header to allow connecting reed switch from +3V3 to BOOT0 pin
Parts:
- J2: footprint Connector_PinHeader_1.27mm:PinHeader_1x07_P1.27mm_Horizontal -> Connector_PinHeader_1.27mm:PinHeader_1x07_P1.27mm_Vertical
- moved J2 7.62 mm to (104.9, 81.2), turned to 0 degrees
Connections:
- J2 pad 1: /BOOT0 -> +3V3
- J2 pad 2: +3V3 -> /SWCLK
- J2 pad 3: /SWCLK -> GND
- J2 pad 4: GND -> /SWDIO
- J2 pad 5: /SWDIO -> /NRST
- J2 pad 6: /NRST -> /SWO
- J2 pad 7: /SWO -> /BOOT0
Routing:
- net /NRST: track 46.8 -> 42.7 mm
- net /SWO: track 22.2 -> 18.1 mm
- net /SWCLK: track 16.1 -> 20.0 mm
- net +3V3: track 47.6 -> 51.0 mm

Commit message: Added additional attenuation functionality for DAC
Parts:
- added R17: 220R, Resistor_SMD:R_0603_1608Metric, F.Cu at (119.8, 103.5)
- moved C12 1.50 mm to (122.8, 103.5)
- moved R4 1.50 mm to (122.8, 102.0)
- moved R2 1.06 mm to (119.8, 102.0), turned to 0 degrees
Connections:
- U2 pad 13: unconnected-(U2-Pad13) -> /GPIO-OD
Routing:
- net /GPIO-OD: track 0.00 -> 3.07 mm
- net Net-(C12-Pad1): track 5.13 -> 7.03 mm
- net GND: track 7.84 -> 9.36 mm

Commit message: Changed R2 to 5.1K to decrease DAC loading and reduce output level for radio microphone input
Parts:
- R2: value 2.2K -> 5.1K
- turned R2 to 180 degrees
Connections:
- R2 pad 1: /AFOUT -> Net-(C12-Pad1)
- R2 pad 2: Net-(C12-Pad1) -> /AFOUT
Changed lines of the file:
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@@
   (net 60 "/GPIO-OD")
   (footprint "Resistor_SMD:R_0603_1608Metric" (layer "F.Cu")
-    (at 119.75 102)
+    (at 119.75 102 180)
     (descr "Resistor SMD 0603 (1608 Metric), square (rectangular) end terminal, IPC_7351 nominal, (Body size source: IPC-SM-782 page 72, https://www.pcb-3d.com/wordpress/wp-content/uploads/ipc-sm-782a_amendment_1_and_2.pdf), generated with kicad-footprint-generator")
     (tags "resistor")
-    (property "LCSC" "C4190")
+    (property "LCSC" "C23186")
     (property "Sheetfile" "File: k1-aioc.kicad_sch")
     (property "Sheetname" "")
@@
       (effects (font (size 0.5 0.5) (thickness 0.1)))
     )
-    (fp_text value "2.2K" (at 0 1.43) (layer "F.Fab")
+    (fp_text value "5.1K" (at 0 1.43) (layer "F.Fab")
       (effects (font (size 1 1) (thickness 0.15)))
     )
@@
     (fp_line (start -0.8 -0.4125) (end 0.8 -0.4125) (layer "F.Fab") (width 0.1))
     (fp_line (start 0.8 -0.4125) (end 0.8 0.4125) (layer "F.Fab") (width 0.1))
-    (pad "1" smd roundrect (at -0.825 0) (size 0.8 0.95) (layers "F.Cu" "F.Paste" "F.Mask") (roundrect_rratio 0.25)
+    (pad "1" smd roundrect (at -0.825 0 180) (size 0.8 0.95) (layers "F.Cu" "F.Paste" "F.Mask") (roundrect_rratio 0.25)
+      (net 32 "Net-(C12-Pad1)") (pintype "passive"))
+    (pad "2" smd roundrect (at 0.825 0 180) (size 0.8 0.95) (layers "F.Cu" "F.Paste" "F.Mask") (roundrect_rratio 0.25)
       (net 45 "/AFOUT") (pintype "passive"))
-    (pad "2" smd roundrect (at 0.825 0) (size 0.8 0.95) (layers "F.Cu" "F.Paste" "F.Mask") (roundrect_rratio 0.25)
-      (net 32 "Net-(C12-Pad1)") (pintype "passive"))
     (model "${KICAD6_3DMODEL_DIR}/Resistor_SMD.3dshapes/R_0603_1608Metric.wrl"
       (offset (xyz 0 0 0))

Commit message: Changed annotation on programming header
Parts:
- moved J2 7.60 mm to (104.9, 88.8), turned to 180 degrees
Connections:
- net /GPIO-OD renamed /DAC_ATTEN
- J2 pad 1: +3V3 -> /BOOT0
- J2 pad 2: /SWCLK -> /SWO
- J2 pad 3: GND -> /NRST
- J2 pad 5: /NRST -> GND
- J2 pad 6: /SWO -> /SWCLK
- J2 pad 7: /BOOT0 -> +3V3
Changed lines of the file:
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@@
   (net 58 "unconnected-(U2-Pad19)")
   (net 59 "Net-(C5-Pad1)")
-  (net 60 "/GPIO-OD")
+  (net 60 "/DAC_ATTEN")
   (footprint "Resistor_SMD:R_0603_1608Metric" (layer "F.Cu")
     (at 119.75 102 180)
@@
       (net 57 "unconnected-(U2-Pad12)") (pinfunction "PA2") (pintype "bidirectional"))
     (pad "13" smd roundrect (at -2.75 4.1625 90) (size 0.3 1.475) (layers "F.Cu" "F.Paste" "F.Mask") (roundrect_rratio 0.25)
-      (net 60 "/GPIO-OD") (pinfunction "PA3") (pintype "bidirectional"))
+      (net 60 "/DAC_ATTEN") (pinfunction "PA3") (pintype "bidirectional"))
     (pad "14" smd roundrect (at -2.25 4.1625 90) (size 0.3 1.475) (layers "F.Cu" "F.Paste" "F.Mask") (roundrect_rratio 0.25)
       (net 45 "/AFOUT") (pinfunction "PA4") (pintype "bidirectional"))
@@
       (net 32 "Net-(C12-Pad1)") (pintype "passive"))
     (pad "2" smd roundrect (at 0.825 0 180) (size 0.8 0.95) (layers "F.Cu" "F.Paste" "F.Mask") (roundrect_rratio 0.25)
-      (net 60 "/GPIO-OD") (pintype "passive"))
+      (net 60 "/DAC_ATTEN") (pintype "passive"))
     (model "${KICAD6_3DMODEL_DIR}/Resistor_SMD.3dshapes/R_0603_1608Metric.wrl"
       (offset (xyz 0 0 0))
@@
   )
   (footprint "Connector_PinHeader_1.27mm:PinHeader_1x07_P1.27mm_Vertical" (layer "F.Cu")
-    (at 104.925 81.15)
+    (at 104.925 88.75 180)
     (descr "Through hole straight pin header, 1x07, 1.27mm pitch, single row")
     (tags "Through hole pin header THT 1x07 1.27mm single row")
@@
       (effects (font (size 1 1) (thickness 0.15)))
     )
-    (fp_line (start -1.11 -0.76) (end 0 -0.76) (layer "F.SilkS") (width 0.12))
-    (fp_line (start 0.563471 0.76) (end 1.11 0.76) (layer "F.SilkS") (width 0.12))
-    (fp_line (start 0.30753 8.315) (end 1.11 8.315) (layer "F.SilkS") (width 0.12))
-    (fp_line (start -1.11 0) (end -1.11 -0.76) (layer "F.SilkS") (width 0.12))
     (fp_line (start -1.11 0.76) (end -1.11 8.315) (layer "F.SilkS") (width 0.12))
-    (fp_line (start -1.11 8.315) (end -0.30753 8.315) (layer "F.SilkS") (width 0.12))
-    (fp_line (start 1.11 0.76) (end 1.11 8.315) (layer "F.SilkS") (width 0.12))
+    (fp_line (start -1.11 0) (end -1.11 -0.76) (layer "F.SilkS") (width 0.12))
+    (fp_line (start 0.30753 8.315) (end 1.11 8.315) (layer "F.SilkS") (width 0.12))
     (fp_line (start -1.11 0.76) (end -0.563471 0.76) (layer "F.SilkS") (width 0.12))
+    (fp_line (start 0.563471 0.76) (end 1.11 0.76) (layer "F.SilkS") (width 0.12))
+    (fp_line (start 1.11 0.76) (end 1.11 8.315) (layer "F.SilkS") (width 0.12))
+    (fp_line (start -1.11 -0.76) (end 0 -0.76) (layer "F.SilkS") (width 0.12))
+    (fp_line (start -1.11 8.315) (end -0.30753 8.315) (layer "F.SilkS") (width 0.12))
     (fp_line (start 1.55 -1.15) (end -1.55 -1.15) (layer "F.CrtYd") (width 0.05))
-    (fp_line (start -1.55 8.8) (end 1.55 8.8) (layer "F.CrtYd") (width 0.05))
     (fp_line (start -1.55 -1.15) (end -1.55 8.8) (layer "F.CrtYd") (width 0.05))
     (fp_line (start 1.55 8.8) (end 1.55 -1.15) (layer "F.CrtYd") (width 0.05))
+    (fp_line (start -1.55 8.8) (end 1.55 8.8) (layer "F.CrtYd") (width 0.05))
     (fp_line (start 1.05 -0.635) (end 1.05 8.255) (layer "F.Fab") (width 0.1))
-    (fp_line (start -0.525 -0.635) (end 1.05 -0.635) (layer "F.Fab") (width 0.1))
-    (fp_line (start -1.05 -0.11) (end -0.525 -0.635) (layer "F.Fab") (width 0.1))
-    (fp_line (start 1.05 8.255) (end -1.05 8.255) (layer "F.Fab") (width 0.1))
     (fp_line (start -1.05 8.255) (end -1.05 -0.11) (layer "F.Fab") (width 0.1))
-    (pad "1" thru_hole rect (at 0 0) (size 1 1) (drill 0.65) (layers *.Cu *.Mask)
-      (net 28 "+3V3") (pinfunction "Pin_1") (pintype "passive"))
-    (pad "2" thru_hole oval (at 0 1.27) (size 1 1) (drill 0.65) (layers *.Cu *.Mask)
-      (net 12 "/SWCLK") (pinfunction "Pin_2") (pintype "passive"))
-    (pad "3" thru_hole oval (at 0 2.54) (size 1 1) (drill 0.65) (layers *.Cu *.Mask)
-      (net 1 "GND") (pinfunction "Pin_3") (pintype "passive"))
-    (pad "4" thru_hole oval (at 0 3.81) (size 1 1) (drill 0.65) (layers *.Cu *.Mask)
+    (fp_line (start 1.05 8.255) (end -1.05 8.255) (layer "F.Fab") (width 0.1))
+    (fp_line (start -1.05 -0.11) (end -0.525 -0.635) (layer "F.Fab") (width 0.1))
+    (fp_line (start -0.525 -0.635) (end 1.05 -0.635) (layer "F.Fab") (width 0.1))
+    (pad "1" thru_hole rect (at 0 0 180) (size 1 1) (drill 0.65) (layers *.Cu *.Mask)
+      (net 51 "/BOOT0") (pinfunction "Pin_1") (pintype "passive"))
+    (pad "2" thru_hole oval (at 0 1.27 180) (size 1 1) (drill 0.65) (layers *.Cu *.Mask)
+      (net 50 "/SWO") (pinfunction "Pin_2") (pintype "passive"))
+    (pad "3" thru_hole oval (at 0 2.54 180) (size 1 1) (drill 0.65) (layers *.Cu *.Mask)
+      (net 49 "/NRST") (pinfunction "Pin_3") (pintype "passive"))
+    (pad "4" thru_hole oval (at 0 3.81 180) (size 1 1) (drill 0.65) (layers *.Cu *.Mask)
       (net 22 "/SWDIO") (pinfunction "Pin_4") (pintype "passive"))
-    (pad "5" thru_hole oval (at 0 5.08) (size 1 1) (drill 0.65) (layers *.Cu *.Mask)
-      (net 49 "/NRST") (pinfunction "Pin_5") (pintype "passive"))
-    (pad "6" thru_hole oval (at 0 6.35) (size 1 1) (drill 0.65) (layers *.Cu *.Mask)
-      (net 50 "/SWO") (pinfunction "Pin_6") (pintype "passive"))
-    (pad "7" thru_hole oval (at 0 7.62) (size 1 1) (drill 0.65) (layers *.Cu *.Mask)
-      (net 51 "/BOOT0") (pinfunction "Pin_7") (pintype "passive"))
+    (pad "5" thru_hole oval (at 0 5.08 180) (size 1 1) (drill 0.65) (layers *.Cu *.Mask)
+      (net 1 "GND") (pinfunction "Pin_5") (pintype "passive"))
+    (pad "6" thru_hole oval (at 0 6.35 180) (size 1 1) (drill 0.65) (layers *.Cu *.Mask)
+      (net 12 "/SWCLK") (pinfunction "Pin_6") (pintype "passive"))
+    (pad "7" thru_hole oval (at 0 7.62 180) (size 1 1) (drill 0.65) (layers *.Cu *.Mask)
+      (net 28 "+3V3") (pinfunction "Pin_7") (pintype "passive"))
     (model "${KICAD6_3DMODEL_DIR}/Connector_PinHeader_1.27mm.3dshapes/PinHeader_1x07_P1.27mm_Vertical.wrl" hide
       (offset (xyz 0 0 0))
@@
   (gr_line (start 105.9 81.4) (end 105.9 83.5) (layer "B.SilkS") (width 0.15))
   (gr_line (start 106.05 83.5) (end 106.05 81.55) (layer "B.SilkS") (width 0.15))
+  (gr_circle (center 105.75 80.75) (end 105.85 80.75) (layer "F.SilkS") (width 0.2) (fill none))
   (gr_rect (start 117.5 104.5) (end 123 110) (layer "B.Mask") (width 0.15) (fill solid))
   (gr_rect (start 117.5 92.75) (end 123 98.25) (layer "B.Mask") (width 0.15) (fill solid))

Commit message: Changed R17 from 220R to 22R
Parts:
- R17: value 220R -> 22R
Changed lines of the file:
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@@
     (descr "Resistor SMD 0603 (1608 Metric), square (rectangular) end terminal, IPC_7351 nominal, (Body size source: IPC-SM-782 page 72, https://www.pcb-3d.com/wordpress/wp-content/uploads/ipc-sm-782a_amendment_1_and_2.pdf), generated with kicad-footprint-generator")
     (tags "resistor")
-    (property "LCSC" "C22962")
+    (property "LCSC" "C23345")
     (property "Sheetfile" "File: k1-aioc.kicad_sch")
     (property "Sheetname" "")
@@
       (effects (font (size 1 1) (thickness 0.15)))
     )
-    (fp_text value "220R" (at 0 1.43) (layer "F.Fab")
+    (fp_text value "22R" (at 0 1.43) (layer "F.Fab")
       (effects (font (size 1 1) (thickness 0.15)))
     )

Commit message: Changed DAC output resistor divider values to 10K/220R
Parts:
- R17: value 22R -> N.M.
- R2: value 5.1K -> 10K
Changed lines of the file:
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@@
     (descr "Resistor SMD 0603 (1608 Metric), square (rectangular) end terminal, IPC_7351 nominal, (Body size source: IPC-SM-782 page 72, https://www.pcb-3d.com/wordpress/wp-content/uploads/ipc-sm-782a_amendment_1_and_2.pdf), generated with kicad-footprint-generator")
     (tags "resistor")
-    (property "LCSC" "C23186")
+    (property "LCSC" "C25804")
     (property "Sheetfile" "File: k1-aioc.kicad_sch")
     (property "Sheetname" "")
@@
       (effects (font (size 0.5 0.5) (thickness 0.1)))
     )
-    (fp_text value "5.1K" (at 0 1.43) (layer "F.Fab")
+    (fp_text value "10K" (at 0 1.43) (layer "F.Fab")
       (effects (font (size 1 1) (thickness 0.15)))
     )
@@
     (descr "Resistor SMD 0603 (1608 Metric), square (rectangular) end terminal, IPC_7351 nominal, (Body size source: IPC-SM-782 page 72, https://www.pcb-3d.com/wordpress/wp-content/uploads/ipc-sm-782a_amendment_1_and_2.pdf), generated with kicad-footprint-generator")
     (tags "resistor")
-    (property "LCSC" "C23345")
-    (property "Sheetfile" "File: k1-aioc.kicad_sch")
-    (property "Sheetname" "")
-    (attr smd)
+    (property "LCSC" "")
+    (property "Sheetfile" "File: k1-aioc.kicad_sch")
+    (property "Sheetname" "")
+    (attr smd exclude_from_pos_files)
     (fp_text reference "R17" (at 0 -1.43) (layer "F.SilkS") hide
       (effects (font (size 1 1) (thickness 0.15)))
     )
-    (fp_text value "22R" (at 0 1.43) (layer "F.Fab")
-      (effects (font (size 1 1) (thickness 0.15)))
-    )
+    (fp_text value "N.M." (at 0 1.43) (layer "F.Fab")
+      (effects (font (size 1 1) (thickness 0.15)))
+    )

Commit message: Adjusted tooling holes for JLCPCB fab
Parts:
- added H2: ToolingHole, AIOC:TOOLING-HOLE, F.Cu at (104.8, 110.2)
- H1: value MountingHole -> ToolingHole; footprint TestPoint:TestPoint_THTPad_D2.0mm_Drill1.0mm -> AIOC:TOOLING-HOLE
- moved C15 8.17 mm to (104.8, 107.2), turned to 90 degrees
- moved C1 2.00 mm to (107.5, 106.5)
- moved Y1 1.25 mm to (109.2, 109.2)
- moved C2 0.50 mm to (111.0, 106.5)
- moved REF** 0.50 mm to (112.0, 106.2)
Routing:
- net /OSCOUT: track 7.84 -> 8.77 mm
- net /OSCIN: track 10.4 -> 9.62 mm
- net /NRST: track 42.7 -> 43.4 mm, vias 1 -> 2
- net GND: vias 60 -> 62
