File: kicad/k1-aioc/k1-aioc.kicad_sch (KiCad schematic)
At the start: 38 parts, among them J1 12401832E402A, J2 Conn_01x06_Female, Q1 BC847BS, U1 LP2985-3.3, U2 STM32F373CBTx, Y1 8MHz/20pF

Commit message: Added bottom silkscreen annotation
Other:
- title: (none) -> All-In-One-Cable (AIOC)
Changed lines of the file:
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@@
 (kicad_sch (version 20211123) (generator eeschema)
   (paper "A4")
+  (title_block
+    (title "All-In-One-Cable (AIOC)")
+    (rev "0")
+  )
   (junction (at 54.61 45.72) (diameter 0) (color 0 0 0 0)
   )
@@
     (pin "1")
     (pin "2")
+  )
+  (symbol (lib_id "Graphic:Logo_Open_Hardware_Small") (at 185.42 173.99 0) (unit 1)
+    (in_bom yes) (on_board yes) (fields_autoplaced)
+    (property "Reference" "#LOGO1" (id 0) (at 185.42 167.005 0)
+      (effects (font (size 1.27 1.27)) hide)
+    )
+    (property "Value" "Logo_Open_Hardware_Small" (id 1) (at 185.42 179.705 0)
+      (effects (font (size 1.27 1.27)) hide)
+    )
+    (property "Footprint" "" (id 2) (at 185.42 173.99 0)
+      (effects (font (size 1.27 1.27)) hide)
+    )
+    (property "Datasheet" "~" (id 3) (at 185.42 173.99 0)
+      (effects (font (size 1.27 1.27)) hide)
+    )
   )
   (symbol (lib_id "power:+3V3") (at 135.89 24.13 0) (unit 1)
@@
   )
   (symbol_instances
+    (path "/194cfacc-9bae-49a7-8ed3-5423fac30fcd"
+      (reference "#LOGO1") (unit 1) (value "Logo_Open_Hardware_Small") (footprint "")
+    )
     (path "/d85775b9-c4b0-412e-975c-5a6388de237b"
       (reference "#PWR01") (unit 1) (value "GND") (footprint "")

Commit message: Correct JLCPCB part rotations
Parts:
- FB1, FB2: value 742792695 -> 600R@100MHz
Changed lines of the file:
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@@
     (in_bom yes) (on_board yes) (fields_autoplaced)
     (property "Reference" "FB2" (id 0) (at 74.9808 25.4 90))
-    (property "Value" "742792695" (id 1) (at 74.9808 27.94 90))
+    (property "Value" "600R@100MHz" (id 1) (at 74.9808 27.94 90))
     (property "Footprint" "Inductor_SMD:L_0603_1608Metric" (id 2) (at 74.93 31.242 90)
       (effects (font (size 1.27 1.27)) hide)
@@
     (in_bom yes) (on_board yes) (fields_autoplaced)
     (property "Reference" "FB1" (id 0) (at 143.4592 25.4 90))
-    (property "Value" "742792695" (id 1) (at 143.4592 27.94 90))
+    (property "Value" "600R@100MHz" (id 1) (at 143.4592 27.94 90))
     (property "Footprint" "Inductor_SMD:L_0603_1608Metric" (id 2) (at 143.51 34.798 90)
       (effects (font (size 1.27 1.27)) hide)
@@
     )
     (path "/94d477a3-a334-4790-b269-fbd4f184062a"
-      (reference "FB1") (unit 1) (value "742792695") (footprint "Inductor_SMD:L_0603_1608Metric")
+      (reference "FB1") (unit 1) (value "600R@100MHz") (footprint "Inductor_SMD:L_0603_1608Metric")
     )
     (path "/572c2d83-95d1-48d5-b7fa-08a534d26aa7"
-      (reference "FB2") (unit 1) (value "742792695") (footprint "Inductor_SMD:L_0603_1608Metric")
+      (reference "FB2") (unit 1) (value "600R@100MHz") (footprint "Inductor_SMD:L_0603_1608Metric")
     )
     (path "/c5b80805-bc26-457d-a1fd-cf6a8b83ea3f"

Commit message: Changed programming header pinout to ST-Link V2 and added SWO pin
Parts:
- removed J2: Conn_01x06_Female, Connector_PinHeader_1.27mm:PinHeader_1x06_P1.27mm_Horizontal, symbol Connector:Conn_01x06_Female
- added J2: Conn_01x07_Male, Connector_PinHeader_1.27mm:PinHeader_1x07_P1.27mm_Horizontal, symbol Connector:Conn_01x07_Male
Connections:
- net +3V3: now also J2.2 (Pin_2)
- net BOOT0: now also J2.1 (Pin_1)
- net GND: now also J2.4 (Pin_4)
- net NRST: now also J2.6 (Pin_6)
- net SWCLK: now also J2.3 (Pin_3)
- net SWDIO: now also J2.5 (Pin_5)
- net SWO: now also J2.7 (Pin_7)
Other:
- note added: "ST-Link V2 SWD Header"

Commit message: Added missing 1.5K USB pullup resistor
Parts:
- added R1: 1.5K, Resistor_SMD:R_0603_1608Metric, symbol Device:R
Connections:
- net +3V3: now also R1.1
- net USB-DP: now also R1.2
Changed lines of the file:
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@@
   (junction (at 36.83 73.66) (diameter 0) (color 0 0 0 0)
   )
+  (junction (at 59.69 50.8) (diameter 0) (color 0 0 0 0)
+  )
   (junction (at 140.97 72.39) (diameter 0) (color 0 0 0 0)
   )
@@
     (stroke (width 0) (type default) (color 0 0 0 0))
   )
+  (wire (pts (xy 59.69 50.8) (xy 59.69 54.61))
+    (stroke (width 0) (type default) (color 0 0 0 0))
+  )
   (wire (pts (xy 76.2 111.76) (xy 76.2 116.84))
     (stroke (width 0) (type default) (color 0 0 0 0))
@@
     (stroke (width 0) (type default) (color 0 0 0 0))
   )
+  (wire (pts (xy 59.69 50.8) (xy 62.23 50.8))
+    (stroke (width 0) (type default) (color 0 0 0 0))
+  )
   (wire (pts (xy 52.07 40.64) (xy 68.58 40.64))
     (stroke (width 0) (type default) (color 0 0 0 0))
@@
     (stroke (width 0) (type default) (color 0 0 0 0))
   )
-  (wire (pts (xy 54.61 50.8) (xy 62.23 50.8))
+  (wire (pts (xy 54.61 50.8) (xy 59.69 50.8))
+    (stroke (width 0) (type default) (color 0 0 0 0))
+  )
+  (wire (pts (xy 59.69 62.23) (xy 59.69 64.77))
     (stroke (width 0) (type default) (color 0 0 0 0))
   )
@@
     (pin "1")
     (pin "2")
+  )
+  (symbol (lib_id "power:+3V3") (at 59.69 64.77 180) (unit 1)
+    (in_bom yes) (on_board yes)
+    (property "Reference" "#PWR07" (id 0) (at 59.69 60.96 0)
+      (effects (font (size 1.27 1.27)) hide)
+    )
+    (property "Value" "+3V3" (id 1) (at 57.15 68.58 0)
+      (effects (font (size 1.27 1.27)) (justify right))
+    )
+    (property "Footprint" "" (id 2) (at 59.69 64.77 0)
+      (effects (font (size 1.27 1.27)) hide)
+    )
+    (property "Datasheet" "" (id 3) (at 59.69 64.77 0)
+      (effects (font (size 1.27 1.27)) hide)
+    )
+    (pin "1")
   )
   (symbol (lib_id "power:GND") (at 99.06 86.36 0) (mirror y) (unit 1)
@@
     (pin "2")
   )
+  (symbol (lib_id "Device:R") (at 59.69 58.42 180) (unit 1)
+    (in_bom yes) (on_board yes) (fields_autoplaced)
+    (property "Reference" "R1" (id 0) (at 62.23 57.1499 0)
+      (effects (font (size 1.27 1.27)) (justify right))
+    )
+    (property "Value" "1.5K" (id 1) (at 62.23 59.6899 0)
+      (effects (font (size 1.27 1.27)) (justify right))
+    )
+    (property "Footprint" "Resistor_SMD:R_0603_1608Metric" (id 2) (at 61.468 58.42 90)
+      (effects (font (size 1.27 1.27)) hide)
+    )
+    (property "Datasheet" "~" (id 3) (at 59.69 58.42 0)
+      (effects (font (size 1.27 1.27)) hide)
+    )
+    (property "LCSC" "C22843" (id 4) (at 62.23 57.1499 0)
+      (effects (font (size 1.27 1.27)) hide)
+    )
+    (pin "1")
+    (pin "2")
+  )
   (symbol (lib_id "Device:C") (at 219.71 142.24 90) (unit 1)
     (in_bom yes) (on_board yes) (fields_autoplaced)
@@
       (reference "#PWR06") (unit 1) (value "GND") (footprint "")
     )
+    (path "/093f73e2-acca-4c30-8a22-7418eba63cd1"
+      (reference "#PWR07") (unit 1) (value "+3V3") (footprint "")
+    )
     (path "/237cec46-d0f0-4e50-b9c9-3c03240013c9"
       (reference "#PWR0101") (unit 1) (value "GND") (footprint "")
@@
       (reference "Q1") (unit 2) (value "BC847BS") (footprint "Package_TO_SOT_SMD:SOT-363_SC-70-6")
     )
+    (path "/731ee317-d717-418e-8a38-f6754143172e"
+      (reference "R1") (unit 1) (value "1.5K") (footprint "Resistor_SMD:R_0603_1608Metric")
+    )
     (path "/5d94c761-144d-4672-9330-c6fa3412fb4e"

Commit message: Added missing biasing resistor on AFIN
Parts:
- added R16: 5.1K, Resistor_SMD:R_0603_1608Metric, symbol Device:R
- R3: value 2.2K -> 5.1K; LCSC C4190 -> C23186
Connections:
- net +3.3VA: now also R16.1
- net AFIN: now also R16.2
Other:
- moved on the sheet: C11, C12, C13, C14, Q1A, Q1B, R12, R13, R3, R4, R5

Commit message: Slightly added board shape and added 1mm thru-hole
Parts:
- added H1: MountingHole, TestPoint:TestPoint_THTPad_D2.0mm_Drill1.0mm, symbol Mechanical:MountingHole
Changed lines of the file:
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@@
     (pin "1")
+  )
+  (symbol (lib_id "Mechanical:MountingHole") (at 19.05 190.5 0) (unit 1)
+    (in_bom yes) (on_board yes) (fields_autoplaced)
+    (property "Reference" "H1" (id 0) (at 21.59 189.2299 0)
+      (effects (font (size 1.27 1.27)) (justify left))
+    )
+    (property "Value" "MountingHole" (id 1) (at 21.59 191.7699 0)
+      (effects (font (size 1.27 1.27)) (justify left))
+    )
+    (property "Footprint" "TestPoint:TestPoint_THTPad_D2.0mm_Drill1.0mm" (id 2) (at 19.05 190.5 0)
+      (effects (font (size 1.27 1.27)) hide)
+    )
+    (property "Datasheet" "~" (id 3) (at 19.05 190.5 0)
+      (effects (font (size 1.27 1.27)) hide)
+    )
   )
   (symbol (lib_id "power:GND") (at 99.06 86.36 0) (mirror y) (unit 1)
@@
       (reference "FB2") (unit 1) (value "600R@100MHz") (footprint "Inductor_SMD:L_0603_1608Metric")
     )
+    (path "/098bba9b-ee08-4339-943b-7dd4169e891d"
+      (reference "H1") (unit 1) (value "MountingHole") (footprint "TestPoint:TestPoint_THTPad_D2.0mm_Drill1.0mm")
+    )
     (path "/c5b80805-bc26-457d-a1fd-cf6a8b83ea3f"

Commit message: Added alternative LED footprints on bottom side
Parts:
- added D3, D4: N.M., LED_SMD:LED_0603_1608Metric, symbol Device:LED
- D1: value LED -> GREEN
- D2: value LED -> RED
Connections:
- net at D1.1 (K), D2.2 (A), R15.1: now also D3.1 (K), D4.2 (A)
- net at D1.2 (A), D2.1 (K), U2.46 (PB9): now also D3.2 (A), D4.1 (K)
Changed lines of the file:
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@@
   (junction (at 54.61 45.72) (diameter 0) (color 0 0 0 0)
   )
+  (junction (at 152.4 152.4) (diameter 0) (color 0 0 0 0)
+  )
   (junction (at 93.98 33.02) (diameter 0) (color 0 0 0 0)
   )
@@
   (junction (at 59.69 50.8) (diameter 0) (color 0 0 0 0)
   )
+  (junction (at 171.45 162.56) (diameter 0) (color 0 0 0 0)
+  )
   (junction (at 140.97 72.39) (diameter 0) (color 0 0 0 0)
   )
@@
   (junction (at 201.93 142.24) (diameter 0) (color 0 0 0 0)
   )
+  (junction (at 152.4 162.56) (diameter 0) (color 0 0 0 0)
+  )
+  (junction (at 171.45 152.4) (diameter 0) (color 0 0 0 0)
+  )
+  (junction (at 171.45 157.48) (diameter 0) (color 0 0 0 0)
+  )
   (junction (at 129.54 88.9) (diameter 0) (color 0 0 0 0)
   )
@@
   (junction (at 152.4 157.48) (diameter 0) (color 0 0 0 0)
   )
-  (junction (at 165.1 157.48) (diameter 0) (color 0 0 0 0)
-  )
   (junction (at 186.69 142.24) (diameter 0) (color 0 0 0 0)
   )
@@
     (stroke (width 0) (type default) (color 0 0 0 0))
   )
+  (wire (pts (xy 171.45 147.32) (xy 170.18 147.32))
+    (stroke (width 0) (type default) (color 0 0 0 0))
+  )
   (wire (pts (xy 66.04 96.52) (xy 66.04 104.14))
     (stroke (width 0) (type default) (color 0 0 0 0))
@@
     (stroke (width 0) (type default) (color 0 0 0 0))
   )
-  (wire (pts (xy 144.78 166.37) (xy 144.78 160.02))
+  (wire (pts (xy 144.78 173.99) (xy 144.78 160.02))
     (stroke (width 0) (type default) (color 0 0 0 0))
   )
@@
     (stroke (width 0) (type default) (color 0 0 0 0))
   )
+  (wire (pts (xy 170.18 166.37) (xy 171.45 166.37))
+    (stroke (width 0) (type default) (color 0 0 0 0))
+  )
   (wire (pts (xy 236.22 36.83) (xy 257.81 36.83))
     (stroke (width 0) (type default) (color 0 0 0 0))
   )
+  (wire (pts (xy 162.56 166.37) (xy 152.4 166.37))
+    (stroke (width 0) (type default) (color 0 0 0 0))
+  )
   (wire (pts (xy 127 88.9) (xy 127 91.44))
     (stroke (width 0) (type default) (color 0 0 0 0))
   )
-  (wire (pts (xy 165.1 157.48) (xy 171.45 157.48))
-    (stroke (width 0) (type default) (color 0 0 0 0))
-  )
   (wire (pts (xy 96.52 35.56) (xy 93.98 35.56))
     (stroke (width 0) (type default) (color 0 0 0 0))
@@
     (stroke (width 0) (type default) (color 0 0 0 0))
   )
+  (wire (pts (xy 162.56 147.32) (xy 152.4 147.32))
+    (stroke (width 0) (type default) (color 0 0 0 0))
+  )
   (wire (pts (xy 104.14 96.52) (xy 66.04 96.52))
     (stroke (width 0) (type default) (color 0 0 0 0))
@@
     (stroke (width 0) (type default) (color 0 0 0 0))
   )
-  (wire (pts (xy 165.1 152.4) (xy 165.1 157.48))
+  (wire (pts (xy 171.45 152.4) (xy 171.45 157.48))
     (stroke (width 0) (type default) (color 0 0 0 0))
   )
@@
     (stroke (width 0) (type default) (color 0 0 0 0))
   )
+  (wire (pts (xy 171.45 166.37) (xy 171.45 162.56))
+    (stroke (width 0) (type default) (color 0 0 0 0))
+  )
   (wire (pts (xy 121.92 88.9) (xy 124.46 88.9))
     (stroke (width 0) (type default) (color 0 0 0 0))
@@
     (stroke (width 0) (type default) (color 0 0 0 0))
   )
-  (wire (pts (xy 165.1 157.48) (xy 165.1 162.56))
+  (wire (pts (xy 171.45 157.48) (xy 171.45 162.56))
     (stroke (width 0) (type default) (color 0 0 0 0))
   )
@@
     (stroke (width 0) (type default) (color 0 0 0 0))
   )
-  (wire (pts (xy 171.45 157.48) (xy 171.45 166.37))
+  (wire (pts (xy 152.4 166.37) (xy 152.4 162.56))
+    (stroke (width 0) (type default) (color 0 0 0 0))
+  )
+  (wire (pts (xy 173.99 157.48) (xy 173.99 173.99))
     (stroke (width 0) (type default) (color 0 0 0 0))
   )
@@
     (stroke (width 0) (type default) (color 0 0 0 0))
   )
-  (wire (pts (xy 171.45 166.37) (xy 144.78 166.37))
+  (wire (pts (xy 173.99 173.99) (xy 144.78 173.99))
     (stroke (width 0) (type default) (color 0 0 0 0))
   )
@@
     (stroke (width 0) (type default) (color 0 0 0 0))
   )
+  (wire (pts (xy 171.45 152.4) (xy 171.45 147.32))
+    (stroke (width 0) (type default) (color 0 0 0 0))
+  )
   (wire (pts (xy 200.66 90.17) (xy 207.01 90.17))
     (stroke (width 0) (type default) (color 0 0 0 0))
@@
     (stroke (width 0) (type default) (color 0 0 0 0))
   )
-  (wire (pts (xy 162.56 152.4) (xy 165.1 152.4))
+  (wire (pts (xy 162.56 152.4) (xy 171.45 152.4))
     (stroke (width 0) (type default) (color 0 0 0 0))
   )
@@
     (stroke (width 0) (type default) (color 0 0 0 0))
   )
+  (wire (pts (xy 171.45 157.48) (xy 173.99 157.48))
+    (stroke (width 0) (type default) (color 0 0 0 0))
+  )
   (wire (pts (xy 152.4 152.4) (xy 152.4 157.48))
     (stroke (width 0) (type default) (color 0 0 0 0))
@@
     (stroke (width 0) (type default) (color 0 0 0 0))
   )
-  (wire (pts (xy 162.56 162.56) (xy 165.1 162.56))
+  (wire (pts (xy 162.56 162.56) (xy 171.45 162.56))
     (stroke (width 0) (type default) (color 0 0 0 0))
   )
@@
   )
   (wire (pts (xy 38.1 113.03) (xy 50.8 113.03))
+    (stroke (width 0) (type default) (color 0 0 0 0))
+  )
+  (wire (pts (xy 152.4 147.32) (xy 152.4 152.4))
     (stroke (width 0) (type default) (color 0 0 0 0))
   )
@@
     )
     (pin "1")
+  )
+  (symbol (lib_id "Device:LED") (at 166.37 147.32 0) (unit 1)
+    (in_bom yes) (on_board yes)
+    (property "Reference" "D3" (id 0) (at 170.18 143.51 0))
+    (property "Value" "N.M." (id 1) (at 170.18 146.05 0))
+    (property "Footprint" "LED_SMD:LED_0603_1608Metric" (id 2) (at 166.37 147.32 0)
+      (effects (font (size 1.27 1.27)) hide)
+    )
+    (property "Datasheet" "~" (id 3) (at 166.37 147.32 0)
+      (effects (font (size 1.27 1.27)) hide)
+    )
+    (property "LCSC" "" (id 4) (at 164.7825 140.97 0)
+      (effects (font (size 1.27 1.27)) hide)
+    )
+    (pin "1")
+    (pin "2")
   )
   (symbol (lib_id "Device:R") (at 68.58 58.42 180) (unit 1)
@@
     (in_bom yes) (on_board yes) (fields_autoplaced)
     (property "Reference" "D1" (id 0) (at 157.1625 146.05 0))
-    (property "Value" "LED" (id 1) (at 157.1625 148.59 0))
+    (property "Value" "GREEN" (id 1) (at 157.1625 148.59 0))
     (property "Footprint" "LED_SMD:LED_0603_1608Metric" (id 2) (at 158.75 152.4 0)
       (effects (font (size 1.27 1.27)) hide)
@@
     (pin "2")
   )
+  (symbol (lib_id "Device:LED") (at 166.37 166.37 180) (unit 1)
+    (in_bom yes) (on_board yes) (fields_autoplaced)
+    (property "Reference" "D4" (id 0) (at 167.9575 158.75 0))
+    (property "Value" "N.M." (id 1) (at 167.9575 161.29 0))
+    (property "Footprint" "LED_SMD:LED_0603_1608Metric" (id 2) (at 166.37 166.37 0)
+      (effects (font (size 1.27 1.27)) hide)
+    )
+    (property "Datasheet" "~" (id 3) (at 166.37 166.37 0)
+      (effects (font (size 1.27 1.27)) hide)
+    )
+    (property "LCSC" "" (id 4) (at 167.9575 172.72 0)
+      (effects (font (size 1.27 1.27)) hide)
+    )
+    (pin "1")
+    (pin "2")
+  )
   (symbol (lib_id "Regulator_Linear:LP2985-3.3") (at 106.68 35.56 0) (unit 1)
     (in_bom yes) (on_board yes) (fields_autoplaced)
@@
     (in_bom yes) (on_board yes) (fields_autoplaced)
     (property "Reference" "D2" (id 0) (at 160.3375 154.94 0))
-    (property "Value" "LED" (id 1) (at 160.3375 157.48 0))
+    (property "Value" "RED" (id 1) (at 160.3375 157.48 0))
     (property "Footprint" "LED_SMD:LED_0603_1608Metric" (id 2) (at 158.75 162.56 0)
       (effects (font (size 1.27 1.27)) hide)
@@
     )
     (path "/44eaa438-6c06-4723-b7a3-c2f7fc0b787d"
-      (reference "D1") (unit 1) (value "LED") (footprint "LED_SMD:LED_0603_1608Metric")
+      (reference "D1") (unit 1) (value "GREEN") (footprint "LED_SMD:LED_0603_1608Metric")
     )
     (path "/b6992821-46a4-4969-b8b4-0f42acce022a"
-      (reference "D2") (unit 1) (value "LED") (footprint "LED_SMD:LED_0603_1608Metric")
+      (reference "D2") (unit 1) (value "RED") (footprint "LED_SMD:LED_0603_1608Metric")
+    )
+    (path "/348f20c8-0ff4-4b81-b8f6-9983a7800ce3"
+      (reference "D3") (unit 1) (value "N.M.") (footprint "LED_SMD:LED_0603_1608Metric")
+    )
+    (path "/accd5217-a765-475c-a33b-d2ad7b0ee6fb"
+      (reference "D4") (unit 1) (value "N.M.") (footprint "LED_SMD:LED_0603_1608Metric")
     )
     (path "/94d477a3-a334-4790-b269-fbd4f184062a"

Commit message: Replaced single 3.3V LDO by dual 3.3V LDO to suppress 1kHz noise from USB in analog signals
Parts:
- removed U1: LP2985-3.3, Package_TO_SOT_SMD:SOT-23-5, symbol Regulator_Linear:LP2985-3.3
- added C5: 4.7u/10V/X5R, Capacitor_SMD:C_0603_1608Metric, symbol Device:C
- added U1: MIC5330-SSYML, Package_DFN_QFN:Micrel_MLF-8-1EP_2x2mm_P0.5mm_EP0.6x1.2mm, symbol aioc:MIC5330-SSYML
- C3: value 10n/NP0 -> 100n; LCSC C57112 -> C14663
- C7: value 100n -> 4.7u/10V/X5R; LCSC C14663 -> C19666
- C9: value 4.7u/10V/X5R -> 100n; LCSC C19666 -> C14663
Connections:
- net +3.3VA: now also FB1.1; no longer FB1.2
- net +3V3: now also U2.1 (VBAT), U1.8 (VOUT1); no longer FB1.1
- net GND: now also C5.2, U1.2 (GND), U1.9 (GND)
- net VIN: now also U1.1 (VIN), U1.4 (EN2), U1.5 (EN1)
- net at C3.1: now also U1.3 (BYP)
- new net: C5.1, FB1.2, U1.7 (VOUT2)
Other:
- moved on the sheet: C4
