File: kicad/k1-aioc/k1-aioc.kicad_sch (KiCad schematic)
At the start: 44 parts, among them J1 12401832E402A, J2 Conn_01x07_Male, Q1 BC847BS, U1 MIC5330-SSYML, U2 STM32F373CBTx, Y1 8MHz/20pF

Commit message: Rotated SWD header to allow connecting reed switch from +3V3 to BOOT0 pin
Parts:
- J2: footprint Connector_PinHeader_1.27mm:PinHeader_1x07_P1.27mm_Horizontal -> Connector_PinHeader_1.27mm:PinHeader_1x07_P1.27mm_Vertical
Connections:
- net +3V3: now also J2.1 (Pin_1); no longer J2.2 (Pin_2)
- net BOOT0: now also J2.7 (Pin_7); no longer J2.1 (Pin_1)
- net GND: now also J2.3 (Pin_3); no longer J2.4 (Pin_4)
- net NRST: now also J2.5 (Pin_5); no longer J2.6 (Pin_6)
- net SWCLK: now also J2.2 (Pin_2); no longer J2.3 (Pin_3)
- net SWDIO: now also J2.4 (Pin_4); no longer J2.5 (Pin_5)
- net SWO: now also J2.6 (Pin_6); no longer J2.7 (Pin_7)
Other:
- note added: "STM Disco SWD Header"
- note removed: "ST-Link V2 SWD Header"
- moved on the sheet: J2
Changed lines of the file:
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@@
     (stroke (width 0) (type default) (color 0 0 0 0))
   )
-  (polyline (pts (xy 31.75 113.03) (xy 29.21 113.03))
-    (stroke (width 0) (type default) (color 0 0 0 0))
-  )
-  (polyline (pts (xy 31.75 116.84) (xy 29.21 116.84))
+  (polyline (pts (xy 22.86 115.57) (xy 19.05 115.57))
     (stroke (width 0) (type default) (color 0 0 0 0))
   )
@@
     (stroke (width 0) (type default) (color 0 0 0 0))
   )
-  (polyline (pts (xy 29.21 116.84) (xy 29.21 128.27))
+  (polyline (pts (xy 29.21 115.57) (xy 29.21 128.27))
     (stroke (width 0) (type default) (color 0 0 0 0))
   )
@@
     (stroke (width 0) (type default) (color 0 0 0 0))
   )
-  (polyline (pts (xy 29.21 115.57) (xy 31.75 115.57))
+  (polyline (pts (xy 19.05 130.81) (xy 31.75 130.81))
     (stroke (width 0) (type default) (color 0 0 0 0))
   )
@@
     (stroke (width 0) (type default) (color 0 0 0 0))
   )
-  (polyline (pts (xy 29.21 113.03) (xy 29.21 115.57))
+  (polyline (pts (xy 19.05 115.57) (xy 19.05 130.81))
     (stroke (width 0) (type default) (color 0 0 0 0))
   )
@@
   )
   (wire (pts (xy 96.52 38.1) (xy 93.98 38.1))
+    (stroke (width 0) (type default) (color 0 0 0 0))
+  )
+  (polyline (pts (xy 29.21 115.57) (xy 31.75 115.57))
     (stroke (width 0) (type default) (color 0 0 0 0))
   )
@@
     (stroke (width 0) (type default) (color 0 0 0 0))
   )
-  (wire (pts (xy 38.1 113.03) (xy 50.8 113.03))
+  (wire (pts (xy 38.1 130.81) (xy 50.8 130.81))
     (stroke (width 0) (type default) (color 0 0 0 0))
   )
@@
     (stroke (width 0) (type default) (color 0 0 0 0))
   )
-  (text "ST-Link V2\nSWD Header" (at 13.97 125.73 0)
-    (effects (font (size 1.27 1.27)) (justify left bottom))
-  )
-  (text "Short Pins for\nBootloader" (at 13.97 116.84 0)
+  (text "STM Disco\nSWD Header" (at 27.94 127 90)
+    (effects (font (size 1.27 1.27)) (justify left bottom))
+  )
+  (text "Short Pins for\nBootloader" (at 17.78 129.54 90)
     (effects (font (size 1.27 1.27)) (justify left bottom))
   )
@@
     (effects (font (size 1.27 1.27)) (justify left bottom))
   )
-  (label "BOOT0" (at 46.99 113.03 0)
+  (label "BOOT0" (at 46.99 130.81 0)
     (effects (font (size 1.27 1.27)) (justify left bottom))
   )
@@
     (pin "2")
   )
-  (symbol (lib_id "Connector:Conn_01x07_Male") (at 33.02 120.65 0) (unit 1)
-    (in_bom yes) (on_board yes) (fields_autoplaced)
-    (property "Reference" "J2" (id 0) (at 33.655 107.95 0))
-    (property "Value" "Conn_01x07_Male" (id 1) (at 33.655 110.49 0))
-    (property "Footprint" "Connector_PinHeader_1.27mm:PinHeader_1x07_P1.27mm_Horizontal" (id 2) (at 33.02 120.65 0)
-      (effects (font (size 1.27 1.27)) hide)
-    )
-    (property "Datasheet" "~" (id 3) (at 33.02 120.65 0)
+  (symbol (lib_id "Connector:Conn_01x07_Male") (at 33.02 123.19 0) (unit 1)
+    (in_bom yes) (on_board yes)
+    (property "Reference" "J2" (id 0) (at 36.83 138.43 0)
+      (effects (font (size 1.27 1.27)) (justify right))
+    )
+    (property "Value" "Conn_01x07_Male" (id 1) (at 36.83 135.89 0)
+      (effects (font (size 1.27 1.27)) (justify right))
+    )
+    (property "Footprint" "Connector_PinHeader_1.27mm:PinHeader_1x07_P1.27mm_Vertical" (id 2) (at 33.02 123.19 0)
+      (effects (font (size 1.27 1.27)) hide)
+    )
+    (property "Datasheet" "~" (id 3) (at 33.02 123.19 0)
       (effects (font (size 1.27 1.27)) hide)
     )
@@
     )
     (path "/f2c9e50d-789f-4fc9-bf13-807bdf38a185"
-      (reference "J2") (unit 1) (value "Conn_01x07_Male") (footprint "Connector_PinHeader_1.27mm:PinHeader_1x07_P1.27mm_Horizontal")
+      (reference "J2") (unit 1) (value "Conn_01x07_Male") (footprint "Connector_PinHeader_1.27mm:PinHeader_1x07_P1.27mm_Vertical")
     )
     (path "/65a95da7-4f7f-4162-9b7a-05aaa141d8aa"

Commit message: Added additional attenuation functionality for DAC
Parts:
- added R17: 220R, Resistor_SMD:R_0603_1608Metric, symbol Device:R
Connections:
- net GPIO-OD: now reaches U2.13 (PA3)
- net GPIO-OD: now also R17.2
- net at C12.1, C13.1, R2.2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: now also R17.1
Other:
- note added: "DAC_ATTEN"
Changed lines of the file:
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@@
   (junction (at 83.82 149.86) (diameter 0) (color 0 0 0 0)
   )
+  (junction (at 200.66 104.14) (diameter 0) (color 0 0 0 0)
+  )
   (junction (at 143.51 33.02) (diameter 0) (color 0 0 0 0)
   )
@@
     (stroke (width 0) (type default) (color 0 0 0 0))
   )
-  (wire (pts (xy 200.66 106.68) (xy 200.66 90.17))
+  (wire (pts (xy 200.66 106.68) (xy 200.66 104.14))
     (stroke (width 0) (type default) (color 0 0 0 0))
   )
@@
     (stroke (width 0) (type default) (color 0 0 0 0))
   )
+  (wire (pts (xy 187.96 104.14) (xy 200.66 104.14))
+    (stroke (width 0) (type default) (color 0 0 0 0))
+  )
+  (wire (pts (xy 200.66 104.14) (xy 200.66 90.17))
+    (stroke (width 0) (type default) (color 0 0 0 0))
+  )
   (wire (pts (xy 83.82 137.16) (xy 104.14 137.16))
     (stroke (width 0) (type default) (color 0 0 0 0))
@@
   )
   (wire (pts (xy 121.92 72.39) (xy 121.92 88.9))
+    (stroke (width 0) (type default) (color 0 0 0 0))
+  )
+  (wire (pts (xy 139.7 104.14) (xy 180.34 104.14))
     (stroke (width 0) (type default) (color 0 0 0 0))
   )
@@
     (effects (font (size 1.27 1.27)) (justify left bottom))
   )
+  (text "DAC_ATTEN" (at 160.02 104.14 0)
+    (effects (font (size 1.27 1.27)) (justify left bottom))
+  )
   (text "Compatible to \nSTM32F302CBTx (no DS-ADC)" (at 129.54 179.07 0)
     (effects (font (size 1.27 1.27)) (justify left bottom))
@@
   )
   (label "RADIO-SPK" (at 238.76 142.24 0)
+    (effects (font (size 1.27 1.27)) (justify left bottom))
+  )
+  (label "GPIO-OD" (at 142.24 104.14 0)
     (effects (font (size 1.27 1.27)) (justify left bottom))
   )
@@
   (symbol (lib_id "Device:R") (at 184.15 106.68 90) (unit 1)
     (in_bom yes) (on_board yes)
-    (property "Reference" "R2" (id 0) (at 180.34 104.14 90))
-    (property "Value" "2.2K" (id 1) (at 185.42 104.14 90))
+    (property "Reference" "R2" (id 0) (at 180.34 109.22 90))
+    (property "Value" "2.2K" (id 1) (at 185.42 109.22 90))
     (property "Footprint" "Resistor_SMD:R_0603_1608Metric" (id 2) (at 184.15 108.458 90)
       (effects (font (size 1.27 1.27)) hide)
@@
     )
     (property "LCSC" "C23186" (id 4) (at 199.39 135.8901 0)
+      (effects (font (size 1.27 1.27)) hide)
+    )
+    (pin "1")
+    (pin "2")
+  )
+  (symbol (lib_id "Device:R") (at 184.15 104.14 270) (unit 1)
+    (in_bom yes) (on_board yes)
+    (property "Reference" "R17" (id 0) (at 180.34 101.6 90))
+    (property "Value" "220R" (id 1) (at 185.42 101.6 90))
+    (property "Footprint" "Resistor_SMD:R_0603_1608Metric" (id 2) (at 184.15 102.362 90)
+      (effects (font (size 1.27 1.27)) hide)
+    )
+    (property "Datasheet" "~" (id 3) (at 184.15 104.14 0)
+      (effects (font (size 1.27 1.27)) hide)
+    )
+    (property "LCSC" "C22962" (id 4) (at 182.8799 101.6 0)
       (effects (font (size 1.27 1.27)) hide)
     )
@@
       (reference "R16") (unit 1) (value "5.1K") (footprint "Resistor_SMD:R_0603_1608Metric")
     )
+    (path "/a6419fd5-a3bc-45f3-9096-0527cd8be825"
+      (reference "R17") (unit 1) (value "220R") (footprint "Resistor_SMD:R_0603_1608Metric")
+    )
     (path "/6928eae3-04b8-42b2-8f00-ec0b9aa50ceb"

Commit message: Changed R2 to 5.1K to decrease DAC loading and reduce output level for radio microphone input
Parts:
- R2: value 2.2K -> 5.1K; LCSC C4190 -> C23186
Connections:
- net AFOUT: now also R2.2; no longer R2.1
- net at C12.1, C13.1, R17.1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: now also R2.1; no longer R2.2
Changed lines of the file:
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@@
     (pin "1")
-  )
-  (symbol (lib_id "Device:R") (at 184.15 106.68 90) (unit 1)
-    (in_bom yes) (on_board yes)
-    (property "Reference" "R2" (id 0) (at 180.34 109.22 90))
-    (property "Value" "2.2K" (id 1) (at 185.42 109.22 90))
-    (property "Footprint" "Resistor_SMD:R_0603_1608Metric" (id 2) (at 184.15 108.458 90)
-      (effects (font (size 1.27 1.27)) hide)
-    )
-    (property "Datasheet" "~" (id 3) (at 184.15 106.68 0)
-      (effects (font (size 1.27 1.27)) hide)
-    )
-    (property "LCSC" "C4190" (id 4) (at 180.34 109.22 0)
-      (effects (font (size 1.27 1.27)) hide)
-    )
-    (pin "1")
-    (pin "2")
   )
   (symbol (lib_id "Device:R") (at 232.41 36.83 270) (unit 1)
@@
     )
     (pin "1")
+  )
+  (symbol (lib_id "Device:R") (at 184.15 106.68 270) (unit 1)
+    (in_bom yes) (on_board yes)
+    (property "Reference" "R2" (id 0) (at 180.34 109.22 90))
+    (property "Value" "5.1K" (id 1) (at 185.42 109.22 90))
+    (property "Footprint" "Resistor_SMD:R_0603_1608Metric" (id 2) (at 184.15 104.902 90)
+      (effects (font (size 1.27 1.27)) hide)
+    )
+    (property "Datasheet" "~" (id 3) (at 184.15 106.68 0)
+      (effects (font (size 1.27 1.27)) hide)
+    )
+    (property "LCSC" "C23186" (id 4) (at 182.8799 104.14 0)
+      (effects (font (size 1.27 1.27)) hide)
+    )
+    (pin "1")
+    (pin "2")
   )
   (symbol (lib_id "Device:R") (at 201.93 134.62 0) (unit 1)
@@
       (reference "R1") (unit 1) (value "1.5K") (footprint "Resistor_SMD:R_0603_1608Metric")
     )
-    (path "/5d94c761-144d-4672-9330-c6fa3412fb4e"
-      (reference "R2") (unit 1) (value "2.2K") (footprint "Resistor_SMD:R_0603_1608Metric")
+    (path "/a395a1f6-0ade-49ae-97ea-2e311cd442a3"
+      (reference "R2") (unit 1) (value "5.1K") (footprint "Resistor_SMD:R_0603_1608Metric")
     )
     (path "/a6e41ec9-f152-4bb3-b386-4a1ce2030945"

Commit message: Changed annotation on programming header
Connections:
- net +3V3: now also J2.7 (Pin_7); no longer J2.1 (Pin_1)
- net BOOT0: now also J2.1 (Pin_1); no longer J2.7 (Pin_7)
- net GND: now also J2.5 (Pin_5); no longer J2.3 (Pin_3)
- net NRST: now also J2.3 (Pin_3); no longer J2.5 (Pin_5)
- net SWCLK: now also J2.6 (Pin_6); no longer J2.2 (Pin_2)
- net SWO: now also J2.2 (Pin_2); no longer J2.6 (Pin_6)
- net GPIO-OD renamed DAC_ATTEN
Other:
- note added: "GPIOA O.D."
- note added: "GPIOA P.P."
- note removed: "DAC_ATTEN"
- note removed: "USART2-RTS"
Changed lines of the file:
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@@
-    (effects (font (size 1.27 1.27)) (justify left bottom))
-  )
-  (text "USART2-RTS" (at 160.02 99.06 0)
     (effects (font (size 1.27 1.27)) (justify left bottom))
   )
@@
     (effects (font (size 1.27 1.27)) (justify left bottom))
   )
+  (text "GPIOA P.P." (at 160.02 99.06 0)
+    (effects (font (size 1.27 1.27)) (justify left bottom))
+  )
   (text "DAC1_OUT1" (at 160.02 106.68 0)
     (effects (font (size 1.27 1.27)) (justify left bottom))
   )
-  (text "DAC_ATTEN" (at 160.02 104.14 0)
+  (text "GPIOA O.D." (at 160.02 104.14 0)
     (effects (font (size 1.27 1.27)) (justify left bottom))
   )
@@
     (effects (font (size 1.27 1.27)) (justify left bottom))
   )
+  (text "GPIOA P.P." (at 160.02 96.52 0)
+    (effects (font (size 1.27 1.27)) (justify left bottom))
+  )
   (label "OSCIN" (at 83.82 134.62 0)
     (effects (font (size 1.27 1.27)) (justify left bottom))
@@
     (effects (font (size 1.27 1.27)) (justify left bottom))
   )
-  (label "GPIO-OD" (at 142.24 104.14 0)
+  (label "DAC_ATTEN" (at 142.24 104.14 0)
     (effects (font (size 1.27 1.27)) (justify left bottom))
   )
@@
     (pin "2")
   )
-  (symbol (lib_id "Connector:Conn_01x07_Male") (at 33.02 123.19 0) (unit 1)
-    (in_bom yes) (on_board yes)
-    (property "Reference" "J2" (id 0) (at 36.83 138.43 0)
-      (effects (font (size 1.27 1.27)) (justify right))
-    )
-    (property "Value" "Conn_01x07_Male" (id 1) (at 36.83 135.89 0)
-      (effects (font (size 1.27 1.27)) (justify right))
-    )
+  (symbol (lib_id "Connector:Conn_01x07_Male") (at 33.02 123.19 0) (mirror x) (unit 1)
+    (in_bom yes) (on_board yes)
+    (property "Reference" "J2" (id 0) (at 36.83 107.95 0)
+      (effects (font (size 1.27 1.27)) (justify right))
+    )
+    (property "Value" "Conn_01x07_Male" (id 1) (at 36.83 110.49 0)
+      (effects (font (size 1.27 1.27)) (justify right))
+    )

Commit message: Changed R17 from 220R to 22R
Parts:
- R17: value 220R -> 22R; LCSC C22962 -> C23345
Changed lines of the file:
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@@
     (pin "1")
+  )
+  (symbol (lib_id "Device:R") (at 184.15 104.14 270) (unit 1)
+    (in_bom yes) (on_board yes)
+    (property "Reference" "R17" (id 0) (at 180.34 101.6 90))
+    (property "Value" "22R" (id 1) (at 185.42 101.6 90))
+    (property "Footprint" "Resistor_SMD:R_0603_1608Metric" (id 2) (at 184.15 102.362 90)
+      (effects (font (size 1.27 1.27)) hide)
+    )
+    (property "Datasheet" "~" (id 3) (at 184.15 104.14 0)
+      (effects (font (size 1.27 1.27)) hide)
+    )
+    (property "LCSC" "C23345" (id 4) (at 184.15 106.68 0)
+      (effects (font (size 1.27 1.27)) hide)
+    )
+    (pin "1")
+    (pin "2")
   )
   (symbol (lib_id "Device:R") (at 147.32 157.48 270) (unit 1)
@@
     (pin "2")
   )
-  (symbol (lib_id "Device:R") (at 184.15 104.14 270) (unit 1)
-    (in_bom yes) (on_board yes)
-    (property "Reference" "R17" (id 0) (at 180.34 101.6 90))
-    (property "Value" "220R" (id 1) (at 185.42 101.6 90))
-    (property "Footprint" "Resistor_SMD:R_0603_1608Metric" (id 2) (at 184.15 102.362 90)
-      (effects (font (size 1.27 1.27)) hide)
-    )
-    (property "Datasheet" "~" (id 3) (at 184.15 104.14 0)
-      (effects (font (size 1.27 1.27)) hide)
-    )
-    (property "LCSC" "C22962" (id 4) (at 182.8799 101.6 0)
-      (effects (font (size 1.27 1.27)) hide)
-    )
-    (pin "1")
-    (pin "2")
-  )
   (symbol (lib_id "Device:R") (at 201.93 149.86 180) (unit 1)
     (in_bom yes) (on_board yes) (fields_autoplaced)
@@
       (reference "R16") (unit 1) (value "5.1K") (footprint "Resistor_SMD:R_0603_1608Metric")
     )
-    (path "/a6419fd5-a3bc-45f3-9096-0527cd8be825"
-      (reference "R17") (unit 1) (value "220R") (footprint "Resistor_SMD:R_0603_1608Metric")
+    (path "/1d2bbe26-fe20-4f5c-9f43-026bf42bc8df"
+      (reference "R17") (unit 1) (value "22R") (footprint "Resistor_SMD:R_0603_1608Metric")
     )
     (path "/6928eae3-04b8-42b2-8f00-ec0b9aa50ceb"

Commit message: Changed DAC output resistor divider values to 10K/220R
Parts:
- R17: value 22R -> N.M.; LCSC C23345 -> (none)
- R2: value 5.1K -> 10K; LCSC C23186 -> C25804
Changed lines of the file:
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@@
     (in_bom yes) (on_board yes)
     (property "Reference" "R17" (id 0) (at 180.34 101.6 90))
-    (property "Value" "22R" (id 1) (at 185.42 101.6 90))
+    (property "Value" "N.M." (id 1) (at 185.42 101.6 90))
     (property "Footprint" "Resistor_SMD:R_0603_1608Metric" (id 2) (at 184.15 102.362 90)
       (effects (font (size 1.27 1.27)) hide)
@@
       (effects (font (size 1.27 1.27)) hide)
     )
-    (property "LCSC" "C23345" (id 4) (at 184.15 106.68 0)
+    (property "LCSC" "" (id 4) (at 184.15 106.68 0)
       (effects (font (size 1.27 1.27)) hide)
     )
@@
     (in_bom yes) (on_board yes)
     (property "Reference" "R2" (id 0) (at 180.34 109.22 90))
-    (property "Value" "5.1K" (id 1) (at 185.42 109.22 90))
+    (property "Value" "10K" (id 1) (at 185.42 109.22 90))
     (property "Footprint" "Resistor_SMD:R_0603_1608Metric" (id 2) (at 184.15 104.902 90)
       (effects (font (size 1.27 1.27)) hide)
@@
       (effects (font (size 1.27 1.27)) hide)
     )
-    (property "LCSC" "C23186" (id 4) (at 182.8799 104.14 0)
+    (property "LCSC" "C25804" (id 4) (at 182.8799 104.14 0)
       (effects (font (size 1.27 1.27)) hide)
     )
@@
     )
     (path "/a395a1f6-0ade-49ae-97ea-2e311cd442a3"
-      (reference "R2") (unit 1) (value "5.1K") (footprint "Resistor_SMD:R_0603_1608Metric")
+      (reference "R2") (unit 1) (value "10K") (footprint "Resistor_SMD:R_0603_1608Metric")
     )
     (path "/a6e41ec9-f152-4bb3-b386-4a1ce2030945"
@@
     )
     (path "/1d2bbe26-fe20-4f5c-9f43-026bf42bc8df"
-      (reference "R17") (unit 1) (value "22R") (footprint "Resistor_SMD:R_0603_1608Metric")
+      (reference "R17") (unit 1) (value "N.M.") (footprint "Resistor_SMD:R_0603_1608Metric")
     )
     (path "/6928eae3-04b8-42b2-8f00-ec0b9aa50ceb"

Commit message: Adjusted tooling holes for JLCPCB fab
Parts:
- added H2: ToolingHole, AIOC:TOOLING-HOLE, symbol Mechanical:MountingHole
- H1: value MountingHole -> ToolingHole; footprint TestPoint:TestPoint_THTPad_D2.0mm_Drill1.0mm -> AIOC:TOOLING-HOLE
Changed lines of the file:
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@@
       (effects (font (size 1.27 1.27)) (justify left))
     )
-    (property "Value" "MountingHole" (id 1) (at 21.59 191.7699 0)
-      (effects (font (size 1.27 1.27)) (justify left))
-    )
-    (property "Footprint" "TestPoint:TestPoint_THTPad_D2.0mm_Drill1.0mm" (id 2) (at 19.05 190.5 0)
+    (property "Value" "ToolingHole" (id 1) (at 21.59 191.7699 0)
+      (effects (font (size 1.27 1.27)) (justify left))
+    )
+    (property "Footprint" "AIOC:TOOLING-HOLE" (id 2) (at 19.05 190.5 0)
       (effects (font (size 1.27 1.27)) hide)
     )
@@
     (pin "2")
   )
+  (symbol (lib_id "Mechanical:MountingHole") (at 39.37 190.5 0) (unit 1)
+    (in_bom yes) (on_board yes) (fields_autoplaced)
+    (property "Reference" "H2" (id 0) (at 41.91 189.2299 0)
+      (effects (font (size 1.27 1.27)) (justify left))
+    )
+    (property "Value" "ToolingHole" (id 1) (at 41.91 191.7699 0)
+      (effects (font (size 1.27 1.27)) (justify left))
+    )
+    (property "Footprint" "AIOC:TOOLING-HOLE" (id 2) (at 39.37 190.5 0)
+      (effects (font (size 1.27 1.27)) hide)
+    )
+    (property "Datasheet" "~" (id 3) (at 39.37 190.5 0)
+      (effects (font (size 1.27 1.27)) hide)
+    )
+  )
   (symbol (lib_id "Device:C") (at 119.38 43.18 0) (mirror y) (unit 1)
     (in_bom yes) (on_board yes) (fields_autoplaced)
@@
     )
     (path "/098bba9b-ee08-4339-943b-7dd4169e891d"
-      (reference "H1") (unit 1) (value "MountingHole") (footprint "TestPoint:TestPoint_THTPad_D2.0mm_Drill1.0mm")
+      (reference "H1") (unit 1) (value "ToolingHole") (footprint "AIOC:TOOLING-HOLE")
+    )
+    (path "/ba24aaa2-cdf6-43f8-bf42-f4a3c365b43c"
+      (reference "H2") (unit 1) (value "ToolingHole") (footprint "AIOC:TOOLING-HOLE")
     )
     (path "/c5b80805-bc26-457d-a1fd-cf6a8b83ea3f"

Commit message: Correct JLCPCB part for green LED
Parts:
- D1: LCSC C72038 -> C72043
Changed lines of the file:
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@@
       (effects (font (size 1.27 1.27)) hide)
     )
-    (property "LCSC" "C72038" (id 4) (at 157.1625 146.05 0)
+    (property "LCSC" "C72043" (id 4) (at 157.1625 146.05 0)
       (effects (font (size 1.27 1.27)) hide)
     )
