File: kicad/k1-aioc/k1-aioc.kicad_sch (KiCad schematic)
At the start: 46 parts, among them J1 12401832E402A, J2 Conn_01x07_Male, Q1 BC847BS, U1 MIC5330-SSYML, U2 STM32F373CBTx, Y1 8MHz/20pF

Commit message: Added missing 3d models
Parts:
- H1, H2: now left out of the parts list
- J1: footprint Connector_USB:USB_C_Receptacle_Amphenol_12401610E4-2A -> AIOC:USB_C_Receptacle_Amphenol_12401832E40-2A
- U1: footprint Package_DFN_QFN:Micrel_MLF-8-1EP_2x2mm_P0.5mm_EP0.6x1.2mm -> AIOC:Micrel_MLF-8-1EP_2x2mm_P0.5mm_EP0.6x1.2mm
- Y1: footprint Crystal:Crystal_SMD_5032-2Pin_5.0x3.2mm -> AIOC:Crystal_SMD_5032-2Pin_5.0x3.2mm
Changed lines of the file:
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@@
   )
   (symbol (lib_id "Mechanical:MountingHole") (at 19.05 190.5 0) (unit 1)
-    (in_bom yes) (on_board yes) (fields_autoplaced)
+    (in_bom no) (on_board yes) (fields_autoplaced)
     (property "Reference" "H1" (id 0) (at 21.59 189.2299 0)
       (effects (font (size 1.27 1.27)) (justify left))
@@
     (property "Reference" "U1" (id 0) (at 106.68 25.4 0))
     (property "Value" "MIC5330-SSYML" (id 1) (at 106.68 27.94 0))
-    (property "Footprint" "Package_DFN_QFN:Micrel_MLF-8-1EP_2x2mm_P0.5mm_EP0.6x1.2mm" (id 2) (at 144.78 41.91 0)
+    (property "Footprint" "AIOC:Micrel_MLF-8-1EP_2x2mm_P0.5mm_EP0.6x1.2mm" (id 2) (at 144.78 41.91 0)
       (effects (font (size 1.27 1.27)) hide)
     )
@@
     (property "Reference" "Y1" (id 0) (at 77.47 142.24 0))
     (property "Value" "8MHz/20pF" (id 1) (at 77.47 144.78 0))
-    (property "Footprint" "Crystal:Crystal_SMD_5032-2Pin_5.0x3.2mm" (id 2) (at 77.47 149.86 0)
+    (property "Footprint" "AIOC:Crystal_SMD_5032-2Pin_5.0x3.2mm" (id 2) (at 77.47 149.86 0)
       (effects (font (size 1.27 1.27)) hide)
     )
@@
   )
   (symbol (lib_id "Mechanical:MountingHole") (at 39.37 190.5 0) (unit 1)
-    (in_bom yes) (on_board yes) (fields_autoplaced)
+    (in_bom no) (on_board yes) (fields_autoplaced)
     (property "Reference" "H2" (id 0) (at 41.91 189.2299 0)
       (effects (font (size 1.27 1.27)) (justify left))
@@
     (property "Reference" "J1" (id 0) (at 36.83 25.4 0))
     (property "Value" "12401832E402A" (id 1) (at 36.83 27.94 0))
-    (property "Footprint" "Connector_USB:USB_C_Receptacle_Amphenol_12401610E4-2A" (id 2) (at 40.64 48.26 0)
+    (property "Footprint" "AIOC:USB_C_Receptacle_Amphenol_12401832E40-2A" (id 2) (at 40.64 48.26 0)
       (effects (font (size 1.27 1.27)) hide)
     )
@@
     )
     (path "/c5b80805-bc26-457d-a1fd-cf6a8b83ea3f"
-      (reference "J1") (unit 1) (value "12401832E402A") (footprint "Connector_USB:USB_C_Receptacle_Amphenol_12401610E4-2A")
+      (reference "J1") (unit 1) (value "12401832E402A") (footprint "AIOC:USB_C_Receptacle_Amphenol_12401832E40-2A")
     )
     (path "/f2c9e50d-789f-4fc9-bf13-807bdf38a185"
@@
     )
     (path "/6928eae3-04b8-42b2-8f00-ec0b9aa50ceb"
-      (reference "U1") (unit 1) (value "MIC5330-SSYML") (footprint "Package_DFN_QFN:Micrel_MLF-8-1EP_2x2mm_P0.5mm_EP0.6x1.2mm")
+      (reference "U1") (unit 1) (value "MIC5330-SSYML") (footprint "AIOC:Micrel_MLF-8-1EP_2x2mm_P0.5mm_EP0.6x1.2mm")
     )
     (path "/374c61ba-2500-40c8-8fa4-5bb019a70699"
@@
     )
     (path "/6f45ce51-4cf6-4c8e-91b8-d0898b19a97d"
-      (reference "Y1") (unit 1) (value "8MHz/20pF") (footprint "Crystal:Crystal_SMD_5032-2Pin_5.0x3.2mm")
-    )
-  )
+      (reference "Y1") (unit 1) (value "8MHz/20pF") (footprint "AIOC:Crystal_SMD_5032-2Pin_5.0x3.2mm")
+    )
+  )

Commit message: Fixed wrong LCSC part definition in sch/pcb
Parts:
- U1: LCSC C3752880 -> C144168
Changed lines of the file:
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@@
       (effects (font (size 1.27 1.27)) hide)
     )
-    (property "LCSC" "C3752880" (id 4) (at 106.68 35.56 0)
+    (property "LCSC" "C144168" (id 4) (at 106.68 35.56 0)
       (effects (font (size 1.27 1.27)) hide)
     )
